Commit message: quadruped start

File: body.urdf (robot description, URDF)
Before this commit: robot robot, 3 links, 2 joints
Links:
- added link BackLowerLeg, mass 1; collision box size=0.2 0.2 1; visual box size=0.2 0.2 1
- added link FrontLowerLeg, mass 1; collision box size=0.2 0.2 1; visual box size=0.2 0.2 1
- added link LeftLeg, mass 1; collision box size=1 0.2 0.2; visual box size=1 0.2 0.2
- added link LeftLowerLeg, mass 1; collision box size=0.2 0.2 1; visual box size=0.2 0.2 1
- added link RightLeg, mass 1; collision box size=1 0.2 0.2; visual box size=1 0.2 0.2
- added link RightLowerLeg, mass 1; collision box size=0.2 0.2 1; visual box size=0.2 0.2 1
- link BackLeg: geometry collision box size=0.2 1 0.2; visual box size=0.2 1 0.2
- link FrontLeg: geometry collision box size=0.2 1 0.2; visual box size=0.2 1 0.2
Joints:
- added joint BackLeg_BackLowerLeg: type revolute, parent BackLeg, child BackLowerLeg, origin xyz=0 -1 0 rpy=0 0 0, axis 1 0 0, limit lower=-3.14159 upper=3.14159 effort=0.0 velocity=0.0
- added joint FrontLeg_FrontLowerLeg: type revolute, parent FrontLeg, child FrontLowerLeg, origin xyz=0 1 0 rpy=0 0 0, axis 1 0 0, limit lower=-3.14159 upper=3.14159 effort=0.0 velocity=0.0
- added joint LeftLeg_LeftLowerLeg: type revolute, parent LeftLeg, child LeftLowerLeg, origin xyz=-1 0 0 rpy=0 0 0, axis 0 1 0, limit lower=-3.14159 upper=3.14159 effort=0.0 velocity=0.0
- added joint RightLeg_RightLowerLeg: type revolute, parent RightLeg, child RightLowerLeg, origin xyz=1 0 0 rpy=0 0 0, axis 0 1 0, limit lower=-3.14159 upper=3.14159 effort=0.0 velocity=0.0
- added joint Torso_LeftLeg: type revolute, parent Torso, child LeftLeg, origin xyz=-0.5 0 1 rpy=0 0 0, axis 0 1 0, limit lower=-3.14159 upper=3.14159 effort=0.0 velocity=0.0
- added joint Torso_RightLeg: type revolute, parent Torso, child RightLeg, origin xyz=0.5 0 1 rpy=0 0 0, axis 0 1 0, limit lower=-3.14159 upper=3.14159 effort=0.0 velocity=0.0
- joint Torso_BackLeg: origin xyz=0.5 0 1.0 rpy=0 0 0 -> xyz=0 -0.5 1 rpy=0 0 0
- joint Torso_FrontLeg: origin xyz=1.5 0 1 rpy=0 0 0 -> xyz=0 0.5 1 rpy=0 0 0

Commit message: assignment 5 done

File: body.urdf (robot description, URDF)
Before this commit: robot robot, 9 links, 8 joints
Links:
- removed link LeftLeg
- removed link LeftLowerLeg
- removed link RightLeg
- removed link RightLowerLeg
- link BackLeg: geometry collision box size=0.5 1 0.5; visual box size=0.5 1 0.5
- link BackLowerLeg: geometry collision box size=0.5 0.5 1; visual box size=0.5 0.5 1
- link FrontLeg: geometry collision box size=0.5 1 0.5; visual box size=0.5 1 0.5
- link FrontLowerLeg: geometry collision box size=0.5 0.5 1; visual box size=0.5 0.5 1
- link Torso: geometry collision box size=1 1 0.5; visual box size=1 1 0.5
Joints:
- removed joint LeftLeg_LeftLowerLeg
- removed joint RightLeg_RightLowerLeg
- removed joint Torso_LeftLeg
- removed joint Torso_RightLeg
- joint Torso_BackLeg: origin xyz=0 -0.5 1 rpy=0 0 0 -> xyz=0 -3.5 1 rpy=0 0 0
- joint Torso_FrontLeg: origin xyz=0 0.5 1 rpy=0 0 0 -> xyz=0 -3.5 1 rpy=0 0 0

Commit message: attempt at a6

File: body.urdf (robot description, URDF)
Before this commit: robot robot, 9 links, 8 joints
Links:
- removed link BackLeg
- removed link BackLowerLeg
- removed link FrontLeg
- removed link FrontLowerLeg
- removed link LeftLeg
- removed link LeftLowerLeg
- removed link RightLeg
- removed link RightLowerLeg
- removed link Torso
- added link 0, mass 1; collision box size=1 1 1; visual box size=1 1 1
- added link 1, mass 1; collision box size=0.2 1 0.2; visual box size=0.2 1 0.2
- added link 2, mass 1; collision box size=0.2 1 0.2; visual box size=0.2 1 0.2
Joints:
- removed joint BackLeg_BackLowerLeg
- removed joint FrontLeg_FrontLowerLeg
- removed joint LeftLeg_LeftLowerLeg
- removed joint RightLeg_RightLowerLeg
- removed joint Torso_BackLeg
- removed joint Torso_FrontLeg
- removed joint Torso_LeftLeg
- removed joint Torso_RightLeg
- added joint 0_1: type revolute, parent 0, child 1, origin xyz=0 -0.5 1 rpy=0 0 0, axis 1 0 0, limit lower=-3.14159 upper=3.14159 effort=0.0 velocity=0.0
- added joint 0_2: type revolute, parent 0, child 2, origin xyz=0 0.5 1 rpy=0 0 0, axis 1 0 0, limit lower=-3.14159 upper=3.14159 effort=0.0 velocity=0.0

Commit message: working through a6

File: body.urdf (robot description, URDF)
Before this commit: robot robot, 9 links, 8 joints
Links:
- removed link BackLeg
- removed link BackLowerLeg
- removed link FrontLeg
- removed link FrontLowerLeg
- removed link LeftLeg
- removed link LeftLowerLeg
- removed link RightLeg
- removed link RightLowerLeg
- removed link Torso
- added link 0, mass 1; collision box size=0.5 0.5 0.5; visual box size=0.5 0.5 0.5
- added link 1, mass 1; collision box size=0.850804977809266 0.10421716389866942 0.7775079972206284; visual box size=0.850804977809266 0.10421716389866942 0.7775079972206284
- added link 2, mass 1; collision box size=0.5333172780788245 0.2647842234465093 0.21970742638097684; visual box size=0.5333172780788245 0.2647842234465093 0.21970742638097684
- added link 3, mass 1; collision box size=0.6879367606864241 0.6344131438540314 0.7231561376522421; visual box size=0.6879367606864241 0.6344131438540314 0.7231561376522421
Joints:
- removed joint BackLeg_BackLowerLeg
- removed joint FrontLeg_FrontLowerLeg
- removed joint LeftLeg_LeftLowerLeg
- removed joint RightLeg_RightLowerLeg
- removed joint Torso_BackLeg
- removed joint Torso_FrontLeg
- removed joint Torso_LeftLeg
- removed joint Torso_RightLeg
- added joint 0_1: type revolute, parent 0, child 1, origin xyz=0 0.25 0.25 rpy=0 0 0, axis 1 0 0, limit lower=-3.14159 upper=3.14159 effort=0.0 velocity=0.0
- added joint 1_2: type revolute, parent 1, child 2, origin xyz=0 0.10421716389866942 0 rpy=0 0 0, axis 1 0 0, limit lower=-3.14159 upper=3.14159 effort=0.0 velocity=0.0
- added joint 2_3: type revolute, parent 2, child 3, origin xyz=0 0.2647842234465093 0 rpy=0 0 0, axis 1 0 0, limit lower=-3.14159 upper=3.14159 effort=0.0 velocity=0.0

Commit message: done with a6

File: body.urdf (robot description, URDF)
Before this commit: robot robot, 4 links, 3 joints
Links:
- added link 4, mass 1; collision box size=0.9862746843308609 0.42137202693752207 0.10060886910344069; visual box size=0.9862746843308609 0.42137202693752207 0.10060886910344069
- link 1: geometry collision box size=0.8781050142563678 0.35903317141996394 0.8447989664456744; visual box size=0.8781050142563678 0.35903317141996394 0.8447989664456744
- link 2: geometry collision box size=0.3461357580185783 0.8226488365179423 0.7007408405805434; visual box size=0.3461357580185783 0.8226488365179423 0.7007408405805434
- link 3: geometry collision box size=0.7547689008005684 0.9827074781539318 0.9411933993905301; visual box size=0.7547689008005684 0.9827074781539318 0.9411933993905301
Joints:
- added joint 3_4: type revolute, parent 3, child 4, origin xyz=0 0.9827074781539318 0 rpy=0 0 0, axis 1 0 0, limit lower=-3.14159 upper=3.14159 effort=0.0 velocity=0.0
- joint 1_2: origin xyz=0 0.10421716389866942 0 rpy=0 0 0 -> xyz=0 0.35903317141996394 0 rpy=0 0 0
- joint 2_3: origin xyz=0 0.2647842234465093 0 rpy=0 0 0 -> xyz=0 0.8226488365179423 0 rpy=0 0 0

Commit message: idk

File: body.urdf (robot description, URDF)
Before this commit: robot robot, 5 links, 4 joints
Links:
- removed link 3
- removed link 4
- link 1: geometry collision box size=0.2269735041100568 0.6867424469304112 0.8816508053086518; visual box size=0.2269735041100568 0.6867424469304112 0.8816508053086518
- link 2: geometry collision box size=0.3488009003294025 0.9900206980394742 0.02875325384663474; visual box size=0.3488009003294025 0.9900206980394742 0.02875325384663474
Joints:
- removed joint 2_3
- removed joint 3_4
- joint 1_2: origin xyz=0 0.35903317141996394 0 rpy=0 0 0 -> xyz=0 0.6867424469304112 0 rpy=0 0 0

Commit message: ok ;

File: body.urdf (robot description, URDF)
Before this commit: robot robot, 3 links, 2 joints
Links:
- added link 3, mass 1; collision box size=0.5181535214124142 0.10671786534573557 0.9690226512978781; visual box size=0.5181535214124142 0.10671786534573557 0.9690226512978781
- added link 4, mass 1; collision box size=0.22930027600817549 0.60090703156068 0.47360316377224265; visual box size=0.22930027600817549 0.60090703156068 0.47360316377224265
- added link 5, mass 1; collision box size=0.024334640450974887 0.5482285491798438 0.9944216473507095; visual box size=0.024334640450974887 0.5482285491798438 0.9944216473507095
- added link 6, mass 1; collision box size=0.39464607038132005 0.9740191460345806 0.3962514349159174; visual box size=0.39464607038132005 0.9740191460345806 0.3962514349159174
- added link 7, mass 1; collision box size=0.9090289043218858 0.9581143334349366 0.8206771705094027; visual box size=0.9090289043218858 0.9581143334349366 0.8206771705094027
- added link 8, mass 1; collision box size=0.9610165701542361 0.0009136659752583265 0.7352395824146539; visual box size=0.9610165701542361 0.0009136659752583265 0.7352395824146539
- added link 9, mass 1; collision box size=0.16014871232857242 0.8660902915402436 0.26036128033551253; visual box size=0.16014871232857242 0.8660902915402436 0.26036128033551253
- link 1: geometry collision box size=0.7506142004594561 0.7850733493913309 0.10285344015999465; visual box size=0.7506142004594561 0.7850733493913309 0.10285344015999465
- link 2: geometry collision box size=0.7825258047921417 0.8673793058410517 0.47154043578111826; visual box size=0.7825258047921417 0.8673793058410517 0.47154043578111826
Joints:
- added joint 2_3: type revolute, parent 2, child 3, origin xyz=0 0.8673793058410517 0 rpy=0 0 0, axis 1 0 0, limit lower=-3.14159 upper=3.14159 effort=0.0 velocity=0.0
- added joint 3_4: type revolute, parent 3, child 4, origin xyz=0 0.10671786534573557 0 rpy=0 0 0, axis 1 0 0, limit lower=-3.14159 upper=3.14159 effort=0.0 velocity=0.0
- added joint 4_5: type revolute, parent 4, child 5, origin xyz=0 0.60090703156068 0 rpy=0 0 0, axis 1 0 0, limit lower=-3.14159 upper=3.14159 effort=0.0 velocity=0.0
- added joint 5_6: type revolute, parent 5, child 6, origin xyz=0 0.5482285491798438 0 rpy=0 0 0, axis 1 0 0, limit lower=-3.14159 upper=3.14159 effort=0.0 velocity=0.0
- added joint 6_7: type revolute, parent 6, child 7, origin xyz=0 0.9740191460345806 0 rpy=0 0 0, axis 1 0 0, limit lower=-3.14159 upper=3.14159 effort=0.0 velocity=0.0
- added joint 7_8: type revolute, parent 7, child 8, origin xyz=0 0.9581143334349366 0 rpy=0 0 0, axis 1 0 0, limit lower=-3.14159 upper=3.14159 effort=0.0 velocity=0.0
- added joint 8_9: type revolute, parent 8, child 9, origin xyz=0 0.0009136659752583265 0 rpy=0 0 0, axis 1 0 0, limit lower=-3.14159 upper=3.14159 effort=0.0 velocity=0.0
- joint 1_2: origin xyz=0 0.6867424469304112 0 rpy=0 0 0 -> xyz=0 0.7850733493913309 0 rpy=0 0 0

Commit message: blocks stil lintersecting

File: body.urdf (robot description, URDF)
Before this commit: robot robot, 10 links, 9 joints
Links:
- removed link 3
- removed link 4
- removed link 5
- removed link 6
- removed link 7
- removed link 8
- removed link 9
- link 1: geometry collision box size=0.8822691445692744 0.21048122739415054 0.35792057917006415; visual box size=0.8822691445692744 0.21048122739415054 0.35792057917006415
- link 2: geometry collision box size=0.7181928846804955 0.9981927364118145 0.20986072012089396; visual box size=0.7181928846804955 0.9981927364118145 0.20986072012089396
Joints:
- removed joint 2_3
- removed joint 3_4
- removed joint 4_5
- removed joint 5_6
- removed joint 6_7
- removed joint 7_8
- removed joint 8_9
- joint 1_2: origin xyz=0 0.7850733493913309 0 rpy=0 0 0 -> xyz=0 -0.21048122739415054 0 rpy=0 0 0

Commit message: done with a7

File: body.urdf (robot description, URDF)
Before this commit: robot robot, 3 links, 2 joints
Links:
- added link 3, mass 1; collision box size=0.29925969187542867 0.9398452833778174 0.6483256295905281; visual box size=0.29925969187542867 0.9398452833778174 0.6483256295905281
- link 1: geometry collision box size=0.001565841814162472 0.1339068170822711 0.21052555552716717; visual box size=0.001565841814162472 0.1339068170822711 0.21052555552716717
- link 2: geometry collision box size=0.04063015313869961 0.38162482358393457 0.3591552103957986; visual box size=0.04063015313869961 0.38162482358393457 0.3591552103957986
Joints:
- added joint 2_3: type revolute, parent 2, child 3, origin xyz=0 0 0.38162482358393457 rpy=0 0 0, axis 1 0 0, limit lower=-3.14159 upper=3.14159 effort=0.0 velocity=0.0
- joint 1_2: origin xyz=0 -0.21048122739415054 0 rpy=0 0 0 -> xyz=0 -0.1339068170822711 0 rpy=0 0 0

Commit message: a8 init

File: body.urdf (robot description, URDF)
Before this commit: robot robot, 4 links, 3 joints
Links:
- added link 4, mass 1; collision box size=0.20783436422886511 0.4474755039578321 0.3069750919214501; visual box size=0.20783436422886511 0.4474755039578321 0.3069750919214501
- added link 5, mass 1; collision box size=0.793172770311626 0.07442780295222307 0.40790467691649557; visual box size=0.793172770311626 0.07442780295222307 0.40790467691649557
- link 1: geometry collision box size=0.21428519745050462 0.22714511763072795 0.2778087203040157; visual box size=0.21428519745050462 0.22714511763072795 0.2778087203040157
- link 2: geometry collision box size=0.29696147984322585 0.4342300469663023 0.33720935639820193; visual box size=0.29696147984322585 0.4342300469663023 0.33720935639820193
- link 3: geometry collision box size=0.21482946918999027 0.3757033863118652 0.4994466899459366; visual box size=0.21482946918999027 0.3757033863118652 0.4994466899459366
Joints:
- added joint 3_4: type revolute, parent 3, child 4, origin xyz=0 0 0.3757033863118652 rpy=0 0 0, axis 1 0 0, limit lower=-3.14159 upper=3.14159 effort=0.0 velocity=0.0
- added joint 4_5: type revolute, parent 4, child 5, origin xyz=0 0 0.4474755039578321 rpy=0 0 0, axis 1 0 0, limit lower=-3.14159 upper=3.14159 effort=0.0 velocity=0.0
- joint 1_2: origin xyz=0 -0.1339068170822711 0 rpy=0 0 0 -> xyz=0 0.22714511763072795 0 rpy=0 0 0
- joint 2_3: origin xyz=0 0 0.38162482358393457 rpy=0 0 0 -> xyz=0 -0.4342300469663023 0 rpy=0 0 0

Commit message: a6

File: body.urdf (robot description, URDF)
Before this commit: robot robot, 5 links, 4 joints
Links:
- link 1: geometry collision box size=0.8865239289829635 0.2112240263500207 0.0571746665611349; visual box size=0.8865239289829635 0.2112240263500207 0.0571746665611349
- link 2: geometry collision box size=0.8116695771452592 0.6785657933039244 0.5549650964993414; visual box size=0.8116695771452592 0.6785657933039244 0.5549650964993414
- link 3: geometry collision box size=0.19021702967088805 0.3032019804924795 0.3256115366170601; visual box size=0.19021702967088805 0.3032019804924795 0.3256115366170601
- link 4: geometry collision box size=0.30717453263971684 0.09876634499843329 0.9244109455478576; visual box size=0.30717453263971684 0.09876634499843329 0.9244109455478576
Joints:
- joint 1_2: origin xyz=0 0.35903317141996394 0 rpy=0 0 0 -> xyz=0 0.2112240263500207 0 rpy=0 0 0
- joint 2_3: origin xyz=0 0.8226488365179423 0 rpy=0 0 0 -> xyz=0 0.6785657933039244 0 rpy=0 0 0
- joint 3_4: origin xyz=0 0.9827074781539318 0 rpy=0 0 0 -> xyz=0 0.3032019804924795 0 rpy=0 0 0

Commit message: okay

File: body.urdf (robot description, URDF)
Before this commit: robot robot, 6 links, 5 joints
Links:
- removed link 2
- removed link 3
- removed link 4
- removed link 5
- link 1: geometry collision box size=0.6600592502132602 0.48398778813771837 0.969725076511445; visual box size=0.6600592502132602 0.48398778813771837 0.969725076511445
Joints:
- removed joint 1_2
- removed joint 2_3
- removed joint 3_4
- removed joint 4_5

Commit message: fixed errors

File: body.urdf (robot description, URDF)
Before this commit: robot robot, 2 links, 1 joints
Links:
- added link 2, mass 1; collision box size=0.8070851615786495 0.6855663700470825 0.9532837591993446; visual box size=0.8070851615786495 0.6855663700470825 0.9532837591993446
- link 0: geometry collision box size=0.25 0.25 0.25; visual box size=0.25 0.25 0.25
- link 1: geometry collision box size=0.3348672089425839 0.2684684119299654 0.22261336100867463; visual box size=0.3348672089425839 0.2684684119299654 0.22261336100867463
Joints:
- added joint 1_2: type revolute, parent 1, child 2, origin xyz=0 0 0.2684684119299654 rpy=0 0 0, axis 1 0 0, limit lower=-3.14159 upper=3.14159 effort=0.0 velocity=0.0

Commit message: working on a8

File: body.urdf (robot description, URDF)
Before this commit: robot robot, 3 links, 2 joints
Links:
- link 1: geometry collision box size=0.3196460997988163 0.21083010640441474 0.3327969110688377; visual box size=0.3196460997988163 0.21083010640441474 0.3327969110688377
- link 2: geometry collision box size=0.7663090141490185 0.24770434761128157 0.8611413077412451; visual box size=0.7663090141490185 0.24770434761128157 0.8611413077412451
Joints:
- joint 1_2: origin xyz=0 0 0.2684684119299654 rpy=0 0 0 -> xyz=0 0 0.21083010640441474 rpy=0 0 0

Commit message: okay

File: body.urdf (robot description, URDF)
Before this commit: robot robot, 5 links, 4 joints
Links:
- added link 5, mass 1; collision box size=0.06457658135637911 0.07958777924060834 0.21158571980446061; visual box size=0.06457658135637911 0.07958777924060834 0.21158571980446061
- added link 6, mass 1; collision box size=0.1421466823246964 0.719455630538323 0.17319493968807664; visual box size=0.1421466823246964 0.719455630538323 0.17319493968807664
- added link 7, mass 1; collision box size=0.10562635018143518 0.956065905675026 0.47326338083017694; visual box size=0.10562635018143518 0.956065905675026 0.47326338083017694
- link 1: geometry collision box size=0.9609976337143882 0.6131635564484855 0.6937235816937284; visual box size=0.9609976337143882 0.6131635564484855 0.6937235816937284
- link 2: geometry collision box size=0.7969028794149656 0.46796953599912117 0.2753105704985277; visual box size=0.7969028794149656 0.46796953599912117 0.2753105704985277
- link 3: geometry collision box size=0.24887140994557644 0.6098014483620026 0.4051958503183193; visual box size=0.24887140994557644 0.6098014483620026 0.4051958503183193
- link 4: geometry collision box size=0.4932883738729279 0.25883323266839986 0.27163989079678474; visual box size=0.4932883738729279 0.25883323266839986 0.27163989079678474
Joints:
- added joint 4_5: type revolute, parent 4, child 5, origin xyz=0 0.25883323266839986 0 rpy=0 0 0, axis 1 0 0, limit lower=-3.14159 upper=3.14159 effort=0.0 velocity=0.0
- added joint 5_6: type revolute, parent 5, child 6, origin xyz=0 0.07958777924060834 0 rpy=0 0 0, axis 1 0 0, limit lower=-3.14159 upper=3.14159 effort=0.0 velocity=0.0
- added joint 6_7: type revolute, parent 6, child 7, origin xyz=0 0.719455630538323 0 rpy=0 0 0, axis 1 0 0, limit lower=-3.14159 upper=3.14159 effort=0.0 velocity=0.0
- joint 1_2: origin xyz=0 0.2112240263500207 0 rpy=0 0 0 -> xyz=0 0.6131635564484855 0 rpy=0 0 0
- joint 2_3: origin xyz=0 0.6785657933039244 0 rpy=0 0 0 -> xyz=0 0.46796953599912117 0 rpy=0 0 0
- joint 3_4: origin xyz=0 0.3032019804924795 0 rpy=0 0 0 -> xyz=0 0.6098014483620026 0 rpy=0 0 0

Commit message: nothing is working

File: body.urdf (robot description, URDF)
Before this commit: robot robot, 9 links, 8 joints
Links:
- removed link BackLeg
- removed link BackLowerLeg
- removed link FrontLeg
- removed link FrontLowerLeg
- removed link LeftLeg
- removed link LeftLowerLeg
- removed link RightLeg
- removed link RightLowerLeg
- added link BackLeft, mass 1; collision box size=0.5 0.5 2; visual box size=0.5 0.5 2
- added link BackRight, mass 1; collision box size=0.5 0.5 2; visual box size=0.5 0.5 2
- link Torso: geometry collision box size=1 3 1; visual box size=1 3 1
Joints:
- removed joint BackLeg_BackLowerLeg
- removed joint FrontLeg_FrontLowerLeg
- removed joint LeftLeg_LeftLowerLeg
- removed joint RightLeg_RightLowerLeg
- removed joint Torso_BackLeg
- removed joint Torso_FrontLeg
- removed joint Torso_LeftLeg
- removed joint Torso_RightLeg
- added joint Torso_BackLeft: type revolute, parent Torso, child BackLeft, origin xyz=0 -1.5 3 rpy=0 0 0, axis 1 0 0, limit lower=-3.14159 upper=3.14159 effort=0.0 velocity=0.0
- added joint Torso_BackRight: type revolute, parent Torso, child BackRight, origin xyz=0 0.5 0 rpy=0 0 0, axis 1 0 0, limit lower=-3.14159 upper=3.14159 effort=0.0 velocity=0.0

Commit message: ugh

File: body.urdf (robot description, URDF)
Before this commit: robot robot, 3 links, 2 joints
Links:
- removed link BackRight
- added link FrontLeg, mass 1; collision box size=0.9559479565570594 1 1; visual box size=0.9559479565570594 1 1
- link BackLeft: geometry collision box size=0.34732967438819556 1 1; visual box size=0.34732967438819556 1 1
- link Torso: geometry collision box size=5 1 1; visual box size=5 1 1
Joints:
- removed joint Torso_BackRight
- added joint Torso_FrontLeg: type revolute, parent Torso, child FrontLeg, origin xyz=1.5 0 1 rpy=0 0 0, axis 1 0 0, limit lower=-3.14159 upper=3.14159 effort=0.0 velocity=0.0
- joint Torso_BackLeft: origin xyz=0 -1.5 3 rpy=0 0 0 -> xyz=0.5 0 1 rpy=0 0 0

Commit message: some progress

File: body.urdf (robot description, URDF)
Before this commit: robot robot, 3 links, 2 joints
Links:
- removed link BackLeft
- removed link FrontLeg
- added link Leg1, mass 1; collision box size=0.8414510005165416 1 1; visual box size=0.8414510005165416 1 1
- added link Leg2, mass 1; collision box size=0.21076834054981736 1 1; visual box size=0.21076834054981736 1 1
- added link Leg3, mass 1; collision box size=0.21076834054981736 1 1; visual box size=0.21076834054981736 1 1
- added link Leg4, mass 1; collision box size=0.21076834054981736 1 1; visual box size=0.21076834054981736 1 1
- added link Leg5, mass 1; collision box size=0.21076834054981736 1 1; visual box size=0.21076834054981736 1 1
- link Torso: geometry collision box size=4 1 1; visual box size=4 1 1
Joints:
- removed joint Torso_BackLeft
- removed joint Torso_FrontLeg
- added joint Torso_Leg1: type revolute, parent Torso, child Leg1, origin xyz=0.5 0 1 rpy=0 0 0, axis 1 0 0, limit lower=-3.14159 upper=3.14159 effort=0.0 velocity=0.0
- added joint Torso_Leg2: type revolute, parent Torso, child Leg2, origin xyz=1.5 0 1 rpy=0 0 0, axis 1 0 0, limit lower=-3.14159 upper=3.14159 effort=0.0 velocity=0.0
- added joint Torso_Leg3: type revolute, parent Torso, child Leg3, origin xyz=0.75 0 1 rpy=0 0 0, axis 1 0 0, limit lower=-3.14159 upper=3.14159 effort=0.0 velocity=0.0
- added joint Torso_Leg4: type revolute, parent Torso, child Leg4, origin xyz=0 0 1 rpy=0 0 0, axis 1 0 0, limit lower=-3.14159 upper=3.14159 effort=0.0 velocity=0.0
- added joint Torso_Leg5: type revolute, parent Torso, child Leg5, origin xyz=2 0 1 rpy=0 0 0, axis 1 0 0, limit lower=-3.14159 upper=3.14159 effort=0.0 velocity=0.0
