Commit message: random stuff working

File: body.urdf (robot description, URDF)
Before this commit: robot robot, 3 links, 2 joints
Links:
- removed link 0
- removed link 1
- removed link 2
- added link Leg1, mass 1; collision box size=0.5515499909444076 1 1; visual box size=0.5515499909444076 1 1
- added link Leg3, mass 1; collision box size=0.42112861190521134 1 1; visual box size=0.42112861190521134 1 1
- added link Leg4, mass 1; collision box size=0.31211953083853383 1 1; visual box size=0.31211953083853383 1 1
- added link Leg5, mass 1; collision box size=0.45710813187582444 1 1; visual box size=0.45710813187582444 1 1
- added link Torso, mass 1; collision box size=4 1 1; visual box size=4 1 1
Joints:
- removed joint 0_1
- removed joint 1_2
- added joint Torso_Leg1: type revolute, parent Torso, child Leg1, origin xyz=0.5 0 1 rpy=0 0 0, axis 1 0 0, limit lower=-3.14159 upper=3.14159 effort=0.0 velocity=0.0
- added joint Torso_Leg3: type revolute, parent Torso, child Leg3, origin xyz=0.75 0 1 rpy=0 0 0, axis 1 0 0, limit lower=-3.14159 upper=3.14159 effort=0.0 velocity=0.0
- added joint Torso_Leg4: type revolute, parent Torso, child Leg4, origin xyz=0 0 1 rpy=0 0 0, axis 1 0 0, limit lower=-3.14159 upper=3.14159 effort=0.0 velocity=0.0
- added joint Torso_Leg5: type revolute, parent Torso, child Leg5, origin xyz=2 0 1 rpy=0 0 0, axis 1 0 0, limit lower=-3.14159 upper=3.14159 effort=0.0 velocity=0.0
