Commit message: things working

File: body0.urdf (robot description, URDF)
Before this commit: robot robot, 3 links, 2 joints
Links:
- added link Leg2, mass 1; collision box size=0.8462496660539656 1 1; visual box size=0.8462496660539656 1 1
- added link Leg3, mass 1; collision box size=0.8857022845809399 1 1; visual box size=0.8857022845809399 1 1
- link Leg1: geometry collision box size=0.4301600452891826 1 1; visual box size=0.4301600452891826 1 1
- link Leg5: geometry collision box size=0.6124516336902097 1 1; visual box size=0.6124516336902097 1 1
Joints:
- added joint Torso_Leg2: type revolute, parent Torso, child Leg2, origin xyz=1.5 0 1 rpy=0 0 0, axis 1 0 0, limit lower=-3.14159 upper=3.14159 effort=0.0 velocity=0.0
- added joint Torso_Leg3: type revolute, parent Torso, child Leg3, origin xyz=0.75 0 1 rpy=0 0 0, axis 1 0 0, limit lower=-3.14159 upper=3.14159 effort=0.0 velocity=0.0

File: body11.urdf (robot description, URDF)
Before this commit: robot robot, 3 links, 2 joints
Links:
- added link Leg2, mass 1; collision box size=0.5814618522574264 1 1; visual box size=0.5814618522574264 1 1
- added link Leg3, mass 1; collision box size=0.8414239228617937 1 1; visual box size=0.8414239228617937 1 1
- link Leg1: geometry collision box size=0.6181977943681362 1 1; visual box size=0.6181977943681362 1 1
- link Leg5: geometry collision box size=0.34772647226887027 1 1; visual box size=0.34772647226887027 1 1
Joints:
- added joint Torso_Leg2: type revolute, parent Torso, child Leg2, origin xyz=1.5 0 1 rpy=0 0 0, axis 1 0 0, limit lower=-3.14159 upper=3.14159 effort=0.0 velocity=0.0
- added joint Torso_Leg3: type revolute, parent Torso, child Leg3, origin xyz=0.75 0 1 rpy=0 0 0, axis 1 0 0, limit lower=-3.14159 upper=3.14159 effort=0.0 velocity=0.0

File: body14.urdf (robot description, URDF)
Before this commit: robot robot, 3 links, 2 joints
Links:
- link Leg1: geometry collision box size=0.937093847422273 1 1; visual box size=0.937093847422273 1 1
- link Leg5: geometry collision box size=0.9428941471888461 1 1; visual box size=0.9428941471888461 1 1

File: body17.urdf (robot description, URDF)
Before this commit: robot robot, 3 links, 2 joints
Links:
- removed link Leg5
- added link Leg2, mass 1; collision box size=0.898945434851693 1 1; visual box size=0.898945434851693 1 1
- added link Leg3, mass 1; collision box size=0.6012074409562733 1 1; visual box size=0.6012074409562733 1 1
- link Leg1: geometry collision box size=0.8455799891088651 1 1; visual box size=0.8455799891088651 1 1
Joints:
- removed joint Torso_Leg5
- added joint Torso_Leg2: type revolute, parent Torso, child Leg2, origin xyz=1.5 0 1 rpy=0 0 0, axis 1 0 0, limit lower=-3.14159 upper=3.14159 effort=0.0 velocity=0.0
- added joint Torso_Leg3: type revolute, parent Torso, child Leg3, origin xyz=0.75 0 1 rpy=0 0 0, axis 1 0 0, limit lower=-3.14159 upper=3.14159 effort=0.0 velocity=0.0

File: body18.urdf (robot description, URDF)
Before this commit: robot robot, 3 links, 2 joints
Links:
- added link Leg3, mass 1; collision box size=0.5401381677110383 1 1; visual box size=0.5401381677110383 1 1
- link Leg1: geometry collision box size=0.2608651353753918 1 1; visual box size=0.2608651353753918 1 1
- link Leg5: geometry collision box size=0.4705939183729781 1 1; visual box size=0.4705939183729781 1 1
Joints:
- added joint Torso_Leg3: type revolute, parent Torso, child Leg3, origin xyz=0.75 0 1 rpy=0 0 0, axis 1 0 0, limit lower=-3.14159 upper=3.14159 effort=0.0 velocity=0.0

File: body2.urdf (robot description, URDF)
Before this commit: robot robot, 3 links, 2 joints
Links:
- added link Leg3, mass 1; collision box size=0.5539073729015156 1 1; visual box size=0.5539073729015156 1 1
- link Leg1: geometry collision box size=0.9784508673228187 1 1; visual box size=0.9784508673228187 1 1
- link Leg5: geometry collision box size=0.5848345073448404 1 1; visual box size=0.5848345073448404 1 1
Joints:
- added joint Torso_Leg3: type revolute, parent Torso, child Leg3, origin xyz=0.75 0 1 rpy=0 0 0, axis 1 0 0, limit lower=-3.14159 upper=3.14159 effort=0.0 velocity=0.0

File: body22.urdf (robot description, URDF)
Before this commit: robot robot, 3 links, 2 joints
Links:
- added link Leg3, mass 1; collision box size=0.8058526225569176 1 1; visual box size=0.8058526225569176 1 1
- added link Leg4, mass 1; collision box size=0.6212187688323089 1 1; visual box size=0.6212187688323089 1 1
- link Leg1: geometry collision box size=0.3910754351263472 1 1; visual box size=0.3910754351263472 1 1
- link Leg5: geometry collision box size=0.3266430656663596 1 1; visual box size=0.3266430656663596 1 1
Joints:
- added joint Torso_Leg3: type revolute, parent Torso, child Leg3, origin xyz=0.75 0 1 rpy=0 0 0, axis 1 0 0, limit lower=-3.14159 upper=3.14159 effort=0.0 velocity=0.0
- added joint Torso_Leg4: type revolute, parent Torso, child Leg4, origin xyz=0 0 1 rpy=0 0 0, axis 1 0 0, limit lower=-3.14159 upper=3.14159 effort=0.0 velocity=0.0

File: body23.urdf (robot description, URDF)
Before this commit: robot robot, 3 links, 2 joints
Links:
- added link Leg2, mass 1; collision box size=0.2621675775885156 1 1; visual box size=0.2621675775885156 1 1
- link Leg1: geometry collision box size=0.7651888190808316 1 1; visual box size=0.7651888190808316 1 1
- link Leg5: geometry collision box size=0.3425896707145277 1 1; visual box size=0.3425896707145277 1 1
Joints:
- added joint Torso_Leg2: type revolute, parent Torso, child Leg2, origin xyz=1.5 0 1 rpy=0 0 0, axis 1 0 0, limit lower=-3.14159 upper=3.14159 effort=0.0 velocity=0.0

File: body24.urdf (robot description, URDF)
Before this commit: robot robot, 3 links, 2 joints
Links:
- removed link Leg5
- added link Leg2, mass 1; collision box size=0.8893384240173405 1 1; visual box size=0.8893384240173405 1 1
- link Leg1: geometry collision box size=0.565415580926967 1 1; visual box size=0.565415580926967 1 1
Joints:
- removed joint Torso_Leg5
- added joint Torso_Leg2: type revolute, parent Torso, child Leg2, origin xyz=1.5 0 1 rpy=0 0 0, axis 1 0 0, limit lower=-3.14159 upper=3.14159 effort=0.0 velocity=0.0

File: body25.urdf (robot description, URDF)
Before this commit: robot robot, 3 links, 2 joints
Links:
- added link Leg3, mass 1; collision box size=0.4124221505016046 1 1; visual box size=0.4124221505016046 1 1
- added link Leg4, mass 1; collision box size=0.7832764777631571 1 1; visual box size=0.7832764777631571 1 1
- link Leg1: geometry collision box size=0.6786903620839772 1 1; visual box size=0.6786903620839772 1 1
- link Leg5: geometry collision box size=0.5239179824053688 1 1; visual box size=0.5239179824053688 1 1
Joints:
- added joint Torso_Leg3: type revolute, parent Torso, child Leg3, origin xyz=0.75 0 1 rpy=0 0 0, axis 1 0 0, limit lower=-3.14159 upper=3.14159 effort=0.0 velocity=0.0
- added joint Torso_Leg4: type revolute, parent Torso, child Leg4, origin xyz=0 0 1 rpy=0 0 0, axis 1 0 0, limit lower=-3.14159 upper=3.14159 effort=0.0 velocity=0.0

File: body26.urdf (robot description, URDF)
Before this commit: robot robot, 3 links, 2 joints
Links:
- removed link Leg5
- added link Leg3, mass 1; collision box size=0.7710373474818202 1 1; visual box size=0.7710373474818202 1 1
- added link Leg4, mass 1; collision box size=0.5440729429576443 1 1; visual box size=0.5440729429576443 1 1
- link Leg1: geometry collision box size=0.3643781238885366 1 1; visual box size=0.3643781238885366 1 1
Joints:
- removed joint Torso_Leg5
- added joint Torso_Leg3: type revolute, parent Torso, child Leg3, origin xyz=0.75 0 1 rpy=0 0 0, axis 1 0 0, limit lower=-3.14159 upper=3.14159 effort=0.0 velocity=0.0
- added joint Torso_Leg4: type revolute, parent Torso, child Leg4, origin xyz=0 0 1 rpy=0 0 0, axis 1 0 0, limit lower=-3.14159 upper=3.14159 effort=0.0 velocity=0.0

File: body27.urdf (robot description, URDF)
Before this commit: robot robot, 3 links, 2 joints
Links:
- removed link Leg5
- added link Leg3, mass 1; collision box size=0.22991978631120108 1 1; visual box size=0.22991978631120108 1 1
- added link Leg4, mass 1; collision box size=0.3687773020212115 1 1; visual box size=0.3687773020212115 1 1
- link Leg1: geometry collision box size=0.394677211503831 1 1; visual box size=0.394677211503831 1 1
Joints:
- removed joint Torso_Leg5
- added joint Torso_Leg3: type revolute, parent Torso, child Leg3, origin xyz=0.75 0 1 rpy=0 0 0, axis 1 0 0, limit lower=-3.14159 upper=3.14159 effort=0.0 velocity=0.0
- added joint Torso_Leg4: type revolute, parent Torso, child Leg4, origin xyz=0 0 1 rpy=0 0 0, axis 1 0 0, limit lower=-3.14159 upper=3.14159 effort=0.0 velocity=0.0

File: body28.urdf (robot description, URDF)
Before this commit: robot robot, 3 links, 2 joints
Links:
- removed link Leg5
- added link Leg2, mass 1; collision box size=0.9189887030531627 1 1; visual box size=0.9189887030531627 1 1
- link Leg1: geometry collision box size=0.6386069487664062 1 1; visual box size=0.6386069487664062 1 1
Joints:
- removed joint Torso_Leg5
- added joint Torso_Leg2: type revolute, parent Torso, child Leg2, origin xyz=1.5 0 1 rpy=0 0 0, axis 1 0 0, limit lower=-3.14159 upper=3.14159 effort=0.0 velocity=0.0

File: body29.urdf (robot description, URDF)
Before this commit: robot robot, 3 links, 2 joints
Links:
- removed link Leg5
- added link Leg2, mass 1; collision box size=0.3983649067791293 1 1; visual box size=0.3983649067791293 1 1
- link Leg1: geometry collision box size=0.9485528269005494 1 1; visual box size=0.9485528269005494 1 1
Joints:
- removed joint Torso_Leg5
- added joint Torso_Leg2: type revolute, parent Torso, child Leg2, origin xyz=1.5 0 1 rpy=0 0 0, axis 1 0 0, limit lower=-3.14159 upper=3.14159 effort=0.0 velocity=0.0

File: body3.urdf (robot description, URDF)
Before this commit: robot robot, 3 links, 2 joints
Links:
- removed link Leg5
- added link Leg4, mass 1; collision box size=0.7172452978460795 1 1; visual box size=0.7172452978460795 1 1
- link Leg1: geometry collision box size=0.8800574627669686 1 1; visual box size=0.8800574627669686 1 1
Joints:
- removed joint Torso_Leg5
- added joint Torso_Leg4: type revolute, parent Torso, child Leg4, origin xyz=0 0 1 rpy=0 0 0, axis 1 0 0, limit lower=-3.14159 upper=3.14159 effort=0.0 velocity=0.0

File: body30.urdf (robot description, URDF)
Before this commit: robot robot, 3 links, 2 joints
Links:
- removed link Leg5
- added link Leg2, mass 1; collision box size=0.29122255846226663 1 1; visual box size=0.29122255846226663 1 1
- link Leg1: geometry collision box size=0.7846731594027339 1 1; visual box size=0.7846731594027339 1 1
Joints:
- removed joint Torso_Leg5
- added joint Torso_Leg2: type revolute, parent Torso, child Leg2, origin xyz=1.5 0 1 rpy=0 0 0, axis 1 0 0, limit lower=-3.14159 upper=3.14159 effort=0.0 velocity=0.0

File: body31.urdf (robot description, URDF)
Before this commit: robot robot, 3 links, 2 joints
Links:
- link Leg1: geometry collision box size=0.985234330176042 1 1; visual box size=0.985234330176042 1 1
- link Leg5: geometry collision box size=0.8177461272908608 1 1; visual box size=0.8177461272908608 1 1

File: body32.urdf (robot description, URDF)
Before this commit: robot robot, 3 links, 2 joints
Links:
- removed link Leg5
- added link Leg3, mass 1; collision box size=0.5389465328947713 1 1; visual box size=0.5389465328947713 1 1
- added link Leg4, mass 1; collision box size=0.6960107686863055 1 1; visual box size=0.6960107686863055 1 1
- link Leg1: geometry collision box size=0.95297956151481 1 1; visual box size=0.95297956151481 1 1
Joints:
- removed joint Torso_Leg5
- added joint Torso_Leg3: type revolute, parent Torso, child Leg3, origin xyz=0.75 0 1 rpy=0 0 0, axis 1 0 0, limit lower=-3.14159 upper=3.14159 effort=0.0 velocity=0.0
- added joint Torso_Leg4: type revolute, parent Torso, child Leg4, origin xyz=0 0 1 rpy=0 0 0, axis 1 0 0, limit lower=-3.14159 upper=3.14159 effort=0.0 velocity=0.0

File: body33.urdf (robot description, URDF)
Before this commit: robot robot, 3 links, 2 joints
Links:
- removed link Leg5
- added link Leg2, mass 1; collision box size=0.5372582149524088 1 1; visual box size=0.5372582149524088 1 1
- added link Leg3, mass 1; collision box size=0.4309491751195119 1 1; visual box size=0.4309491751195119 1 1
- link Leg1: geometry collision box size=0.2949924973115867 1 1; visual box size=0.2949924973115867 1 1
Joints:
- removed joint Torso_Leg5
- added joint Torso_Leg2: type revolute, parent Torso, child Leg2, origin xyz=1.5 0 1 rpy=0 0 0, axis 1 0 0, limit lower=-3.14159 upper=3.14159 effort=0.0 velocity=0.0
- added joint Torso_Leg3: type revolute, parent Torso, child Leg3, origin xyz=0.75 0 1 rpy=0 0 0, axis 1 0 0, limit lower=-3.14159 upper=3.14159 effort=0.0 velocity=0.0

File: body34.urdf (robot description, URDF)
Before this commit: robot robot, 3 links, 2 joints
Links:
- removed link Leg5
- added link Leg4, mass 1; collision box size=0.2660725388803393 1 1; visual box size=0.2660725388803393 1 1
- link Leg1: geometry collision box size=0.2573380692284212 1 1; visual box size=0.2573380692284212 1 1
Joints:
- removed joint Torso_Leg5
- added joint Torso_Leg4: type revolute, parent Torso, child Leg4, origin xyz=0 0 1 rpy=0 0 0, axis 1 0 0, limit lower=-3.14159 upper=3.14159 effort=0.0 velocity=0.0
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