Commit message: doing 2

File: body0.urdf (robot description, URDF)
Before this commit: robot robot, 5 links, 4 joints
Links:
- removed link Leg2
- added link Leg4, mass 1; collision box size=0.361179002540301 1 1; visual box size=0.361179002540301 1 1
- link Leg1: geometry collision box size=0.34817342867011325 1 1; visual box size=0.34817342867011325 1 1
- link Leg3: geometry collision box size=0.7411725138342644 1 1; visual box size=0.7411725138342644 1 1
- link Leg5: geometry collision box size=0.727984106167159 1 1; visual box size=0.727984106167159 1 1
Joints:
- removed joint Torso_Leg2
- added joint Torso_Leg4: type revolute, parent Torso, child Leg4, origin xyz=0 0 1 rpy=0 0 0, axis 1 0 0, limit lower=-3.14159 upper=3.14159 effort=0.0 velocity=0.0

File: body1.urdf (robot description, URDF)
Before this commit: robot robot, 6 links, 5 joints
Links:
- link Leg1: geometry collision box size=0.488832179635942 1 1; visual box size=0.488832179635942 1 1
- link Leg2: geometry collision box size=0.4148302955347403 1 1; visual box size=0.4148302955347403 1 1
- link Leg3: geometry collision box size=0.6869298570287079 1 1; visual box size=0.6869298570287079 1 1
- link Leg4: geometry collision box size=0.6229036023501924 1 1; visual box size=0.6229036023501924 1 1
- link Leg5: geometry collision box size=0.7327858416786772 1 1; visual box size=0.7327858416786772 1 1

File: body10.urdf (robot description, URDF)
Before this commit: robot robot, 6 links, 5 joints
Links:
- removed link Leg5
- link Leg1: geometry collision box size=0.9497739962929466 1 1; visual box size=0.9497739962929466 1 1
- link Leg2: geometry collision box size=0.7058541279179662 1 1; visual box size=0.7058541279179662 1 1
- link Leg3: geometry collision box size=0.6720976112396118 1 1; visual box size=0.6720976112396118 1 1
- link Leg4: geometry collision box size=0.6720198649060829 1 1; visual box size=0.6720198649060829 1 1
Joints:
- removed joint Torso_Leg5

File: body11.urdf (robot description, URDF)
Before this commit: robot robot, 5 links, 4 joints
Links:
- removed link Leg2
- removed link Leg3
- removed link Leg5
- added link Leg4, mass 1; collision box size=0.9634878368339403 1 1; visual box size=0.9634878368339403 1 1
- link Leg1: geometry collision box size=0.7050804140999702 1 1; visual box size=0.7050804140999702 1 1
Joints:
- removed joint Torso_Leg2
- removed joint Torso_Leg3
- removed joint Torso_Leg5
- added joint Torso_Leg4: type revolute, parent Torso, child Leg4, origin xyz=0 0 1 rpy=0 0 0, axis 1 0 0, limit lower=-3.14159 upper=3.14159 effort=0.0 velocity=0.0

File: body12.urdf (robot description, URDF)
Before this commit: robot robot, 6 links, 5 joints
Links:
- link Leg1: geometry collision box size=0.7023436635577134 1 1; visual box size=0.7023436635577134 1 1
- link Leg2: geometry collision box size=0.47856701018417436 1 1; visual box size=0.47856701018417436 1 1
- link Leg3: geometry collision box size=0.26595151700123226 1 1; visual box size=0.26595151700123226 1 1
- link Leg4: geometry collision box size=0.23240362927190958 1 1; visual box size=0.23240362927190958 1 1
- link Leg5: geometry collision box size=0.2295520256683161 1 1; visual box size=0.2295520256683161 1 1

File: body13.urdf (robot description, URDF)
Before this commit: robot robot, 6 links, 5 joints
Links:
- removed link Leg3
- removed link Leg5
- link Leg1: geometry collision box size=0.42275615847573234 1 1; visual box size=0.42275615847573234 1 1
- link Leg2: geometry collision box size=0.3706476570035423 1 1; visual box size=0.3706476570035423 1 1
- link Leg4: geometry collision box size=0.9204736914902956 1 1; visual box size=0.9204736914902956 1 1
Joints:
- removed joint Torso_Leg3
- removed joint Torso_Leg5

File: body14.urdf (robot description, URDF)
Before this commit: robot robot, 3 links, 2 joints
Links:
- removed link Leg5
- added link Leg3, mass 1; collision box size=0.7628099682450646 1 1; visual box size=0.7628099682450646 1 1
- added link Leg4, mass 1; collision box size=0.5964766383551799 1 1; visual box size=0.5964766383551799 1 1
- link Leg1: geometry collision box size=0.7774039078443655 1 1; visual box size=0.7774039078443655 1 1
Joints:
- removed joint Torso_Leg5
- added joint Torso_Leg3: type revolute, parent Torso, child Leg3, origin xyz=0.75 0 1 rpy=0 0 0, axis 1 0 0, limit lower=-3.14159 upper=3.14159 effort=0.0 velocity=0.0
- added joint Torso_Leg4: type revolute, parent Torso, child Leg4, origin xyz=0 0 1 rpy=0 0 0, axis 1 0 0, limit lower=-3.14159 upper=3.14159 effort=0.0 velocity=0.0

File: body15.urdf (robot description, URDF)
Before this commit: robot robot, 6 links, 5 joints
Links:
- link Leg1: geometry collision box size=0.6178437032759377 1 1; visual box size=0.6178437032759377 1 1
- link Leg2: geometry collision box size=0.9803468858607434 1 1; visual box size=0.9803468858607434 1 1
- link Leg3: geometry collision box size=0.8759200987065219 1 1; visual box size=0.8759200987065219 1 1
- link Leg4: geometry collision box size=0.9993715815548305 1 1; visual box size=0.9993715815548305 1 1
- link Leg5: geometry collision box size=0.39925020094506664 1 1; visual box size=0.39925020094506664 1 1

File: body16.urdf (robot description, URDF)
Before this commit: robot robot, 6 links, 5 joints
Links:
- removed link Leg2
- removed link Leg5
- link Leg1: geometry collision box size=0.289392921361394 1 1; visual box size=0.289392921361394 1 1
- link Leg3: geometry collision box size=0.2989541324955034 1 1; visual box size=0.2989541324955034 1 1
- link Leg4: geometry collision box size=0.2883376804700765 1 1; visual box size=0.2883376804700765 1 1
Joints:
- removed joint Torso_Leg2
- removed joint Torso_Leg5

File: body17.urdf (robot description, URDF)
Before this commit: robot robot, 4 links, 3 joints
Links:
- added link Leg4, mass 1; collision box size=0.5155317643575572 1 1; visual box size=0.5155317643575572 1 1
- added link Leg5, mass 1; collision box size=0.998805021760844 1 1; visual box size=0.998805021760844 1 1
- link Leg1: geometry collision box size=0.7851265741627007 1 1; visual box size=0.7851265741627007 1 1
- link Leg2: geometry collision box size=0.7449502345719212 1 1; visual box size=0.7449502345719212 1 1
- link Leg3: geometry collision box size=0.26336645049213847 1 1; visual box size=0.26336645049213847 1 1
Joints:
- added joint Torso_Leg4: type revolute, parent Torso, child Leg4, origin xyz=0 0 1 rpy=0 0 0, axis 1 0 0, limit lower=-3.14159 upper=3.14159 effort=0.0 velocity=0.0
- added joint Torso_Leg5: type revolute, parent Torso, child Leg5, origin xyz=2 0 1 rpy=0 0 0, axis 1 0 0, limit lower=-3.14159 upper=3.14159 effort=0.0 velocity=0.0

File: body18.urdf (robot description, URDF)
Before this commit: robot robot, 4 links, 3 joints
Links:
- link Leg1: geometry collision box size=0.25965243358424533 1 1; visual box size=0.25965243358424533 1 1
- link Leg3: geometry collision box size=0.21126537755796254 1 1; visual box size=0.21126537755796254 1 1
- link Leg5: geometry collision box size=0.2042823311371551 1 1; visual box size=0.2042823311371551 1 1

File: body19.urdf (robot description, URDF)
Before this commit: robot robot, 6 links, 5 joints
Links:
- removed link Leg2
- removed link Leg4
- link Leg1: geometry collision box size=0.7089284259257853 1 1; visual box size=0.7089284259257853 1 1
- link Leg3: geometry collision box size=0.9961633276640047 1 1; visual box size=0.9961633276640047 1 1
- link Leg5: geometry collision box size=0.5598457139069741 1 1; visual box size=0.5598457139069741 1 1
Joints:
- removed joint Torso_Leg2
- removed joint Torso_Leg4

File: body2.urdf (robot description, URDF)
Before this commit: robot robot, 4 links, 3 joints
Links:
- removed link Leg5
- added link Leg2, mass 1; collision box size=0.5029761759270952 1 1; visual box size=0.5029761759270952 1 1
- link Leg1: geometry collision box size=0.8611275209555731 1 1; visual box size=0.8611275209555731 1 1
- link Leg3: geometry collision box size=0.9739594508252394 1 1; visual box size=0.9739594508252394 1 1
Joints:
- removed joint Torso_Leg5
- added joint Torso_Leg2: type revolute, parent Torso, child Leg2, origin xyz=1.5 0 1 rpy=0 0 0, axis 1 0 0, limit lower=-3.14159 upper=3.14159 effort=0.0 velocity=0.0

File: body20.urdf (robot description, URDF)
Before this commit: robot robot, 6 links, 5 joints
Links:
- removed link Leg5
- link Leg1: geometry collision box size=0.7428186013923448 1 1; visual box size=0.7428186013923448 1 1
- link Leg2: geometry collision box size=0.869168158360442 1 1; visual box size=0.869168158360442 1 1
- link Leg3: geometry collision box size=0.982361172236049 1 1; visual box size=0.982361172236049 1 1
- link Leg4: geometry collision box size=0.5593573857297987 1 1; visual box size=0.5593573857297987 1 1
Joints:
- removed joint Torso_Leg5

File: body21.urdf (robot description, URDF)
Before this commit: robot robot, 6 links, 5 joints
Links:
- removed link Leg4
- removed link Leg5
- link Leg1: geometry collision box size=0.4725207098130592 1 1; visual box size=0.4725207098130592 1 1
- link Leg2: geometry collision box size=0.3187651626261396 1 1; visual box size=0.3187651626261396 1 1
- link Leg3: geometry collision box size=0.23060421247534393 1 1; visual box size=0.23060421247534393 1 1
Joints:
- removed joint Torso_Leg4
- removed joint Torso_Leg5

File: body22.urdf (robot description, URDF)
Before this commit: robot robot, 5 links, 4 joints
Links:
- removed link Leg4
- link Leg1: geometry collision box size=0.37080394775941833 1 1; visual box size=0.37080394775941833 1 1
- link Leg3: geometry collision box size=0.963573954755452 1 1; visual box size=0.963573954755452 1 1
- link Leg5: geometry collision box size=0.9644992658274496 1 1; visual box size=0.9644992658274496 1 1
Joints:
- removed joint Torso_Leg4

File: body23.urdf (robot description, URDF)
Before this commit: robot robot, 4 links, 3 joints
Links:
- removed link Leg2
- added link Leg3, mass 1; collision box size=0.2846545143151928 1 1; visual box size=0.2846545143151928 1 1
- added link Leg4, mass 1; collision box size=0.5379774747909021 1 1; visual box size=0.5379774747909021 1 1
- link Leg1: geometry collision box size=0.49113566519340585 1 1; visual box size=0.49113566519340585 1 1
- link Leg5: geometry collision box size=0.9130806398942386 1 1; visual box size=0.9130806398942386 1 1
Joints:
- removed joint Torso_Leg2
- added joint Torso_Leg3: type revolute, parent Torso, child Leg3, origin xyz=0.75 0 1 rpy=0 0 0, axis 1 0 0, limit lower=-3.14159 upper=3.14159 effort=0.0 velocity=0.0
- added joint Torso_Leg4: type revolute, parent Torso, child Leg4, origin xyz=0 0 1 rpy=0 0 0, axis 1 0 0, limit lower=-3.14159 upper=3.14159 effort=0.0 velocity=0.0

File: body24.urdf (robot description, URDF)
Before this commit: robot robot, 3 links, 2 joints
Links:
- added link Leg5, mass 1; collision box size=0.2307640252027243 1 1; visual box size=0.2307640252027243 1 1
- link Leg1: geometry collision box size=0.49168500272048093 1 1; visual box size=0.49168500272048093 1 1
- link Leg2: geometry collision box size=0.8476351828340385 1 1; visual box size=0.8476351828340385 1 1
Joints:
- added joint Torso_Leg5: type revolute, parent Torso, child Leg5, origin xyz=2 0 1 rpy=0 0 0, axis 1 0 0, limit lower=-3.14159 upper=3.14159 effort=0.0 velocity=0.0

File: body25.urdf (robot description, URDF)
Before this commit: robot robot, 5 links, 4 joints
Links:
- removed link Leg5
- link Leg1: geometry collision box size=0.3356792805489982 1 1; visual box size=0.3356792805489982 1 1
- link Leg3: geometry collision box size=0.9928345537446539 1 1; visual box size=0.9928345537446539 1 1
- link Leg4: geometry collision box size=0.791150583087979 1 1; visual box size=0.791150583087979 1 1
Joints:
- removed joint Torso_Leg5

File: body26.urdf (robot description, URDF)
Before this commit: robot robot, 4 links, 3 joints
Links:
- removed link Leg3
- link Leg1: geometry collision box size=0.5042266979388504 1 1; visual box size=0.5042266979388504 1 1
- link Leg4: geometry collision box size=0.629007187473735 1 1; visual box size=0.629007187473735 1 1
Joints:
- removed joint Torso_Leg3
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