Commit message: done w a8

File: body0.urdf (robot description, URDF)
Before this commit: robot robot, 5 links, 4 joints
Links:
- removed link Leg4
- removed link Leg5
- link Leg1: geometry collision box size=0.9177311712343135 1 1; visual box size=0.9177311712343135 1 1
- link Leg3: geometry collision box size=0.7648325442321762 1 1; visual box size=0.7648325442321762 1 1
Joints:
- removed joint Torso_Leg4
- removed joint Torso_Leg5

File: body1.urdf (robot description, URDF)
Before this commit: robot robot, 6 links, 5 joints
Links:
- removed link Leg2
- removed link Leg4
- removed link Leg5
- link Leg1: geometry collision box size=0.9291172499932745 1 1; visual box size=0.9291172499932745 1 1
- link Leg3: geometry collision box size=0.7828733845609002 1 1; visual box size=0.7828733845609002 1 1
Joints:
- removed joint Torso_Leg2
- removed joint Torso_Leg4
- removed joint Torso_Leg5

File: body10.urdf (robot description, URDF)
Before this commit: robot robot, 5 links, 4 joints
Links:
- removed link Leg4
- added link Leg5, mass 1; collision box size=0.3618355356486969 1 1; visual box size=0.3618355356486969 1 1
- link Leg1: geometry collision box size=0.5680875959476916 1 1; visual box size=0.5680875959476916 1 1
- link Leg2: geometry collision box size=0.7952926546117152 1 1; visual box size=0.7952926546117152 1 1
- link Leg3: geometry collision box size=0.33769935113355154 1 1; visual box size=0.33769935113355154 1 1
Joints:
- removed joint Torso_Leg4
- added joint Torso_Leg5: type revolute, parent Torso, child Leg5, origin xyz=2 0 1 rpy=0 0 0, axis 1 0 0, limit lower=-3.14159 upper=3.14159 effort=0.0 velocity=0.0

File: body100.urdf (robot description, URDF)
Before this commit: robot robot, 3 links, 2 joints
Links:
- removed link Leg4
- added link Leg2, mass 1; collision box size=0.5203718440584586 1 1; visual box size=0.5203718440584586 1 1
- added link Leg3, mass 1; collision box size=0.3923724151280021 1 1; visual box size=0.3923724151280021 1 1
- added link Leg5, mass 1; collision box size=0.4378861928432938 1 1; visual box size=0.4378861928432938 1 1
- link Leg1: geometry collision box size=0.39795450465291804 1 1; visual box size=0.39795450465291804 1 1
Joints:
- removed joint Torso_Leg4
- added joint Torso_Leg2: type revolute, parent Torso, child Leg2, origin xyz=1.5 0 1 rpy=0 0 0, axis 1 0 0, limit lower=-3.14159 upper=3.14159 effort=0.0 velocity=0.0
- added joint Torso_Leg3: type revolute, parent Torso, child Leg3, origin xyz=0.75 0 1 rpy=0 0 0, axis 1 0 0, limit lower=-3.14159 upper=3.14159 effort=0.0 velocity=0.0
- added joint Torso_Leg5: type revolute, parent Torso, child Leg5, origin xyz=2 0 1 rpy=0 0 0, axis 1 0 0, limit lower=-3.14159 upper=3.14159 effort=0.0 velocity=0.0

File: body1000.urdf (robot description, URDF)
Before this commit: robot robot, 5 links, 4 joints
Links:
- added link Leg2, mass 1; collision box size=0.49347142026094226 1 1; visual box size=0.49347142026094226 1 1
- link Leg1: geometry collision box size=0.36621669222297815 1 1; visual box size=0.36621669222297815 1 1
- link Leg3: geometry collision box size=0.20851126797846167 1 1; visual box size=0.20851126797846167 1 1
- link Leg4: geometry collision box size=0.5358660909193786 1 1; visual box size=0.5358660909193786 1 1
- link Leg5: geometry collision box size=0.9784894519563383 1 1; visual box size=0.9784894519563383 1 1
Joints:
- added joint Torso_Leg2: type revolute, parent Torso, child Leg2, origin xyz=1.5 0 1 rpy=0 0 0, axis 1 0 0, limit lower=-3.14159 upper=3.14159 effort=0.0 velocity=0.0

File: body1001.urdf (robot description, URDF)
Before this commit: robot robot, 3 links, 2 joints
Links:
- added link Leg2, mass 1; collision box size=0.2086866093437151 1 1; visual box size=0.2086866093437151 1 1
- added link Leg4, mass 1; collision box size=0.3182400076705248 1 1; visual box size=0.3182400076705248 1 1
- added link Leg5, mass 1; collision box size=0.47748447735970223 1 1; visual box size=0.47748447735970223 1 1
- link Leg1: geometry collision box size=0.5879749743130238 1 1; visual box size=0.5879749743130238 1 1
- link Leg3: geometry collision box size=0.3860177683273988 1 1; visual box size=0.3860177683273988 1 1
Joints:
- added joint Torso_Leg2: type revolute, parent Torso, child Leg2, origin xyz=1.5 0 1 rpy=0 0 0, axis 1 0 0, limit lower=-3.14159 upper=3.14159 effort=0.0 velocity=0.0
- added joint Torso_Leg4: type revolute, parent Torso, child Leg4, origin xyz=0 0 1 rpy=0 0 0, axis 1 0 0, limit lower=-3.14159 upper=3.14159 effort=0.0 velocity=0.0
- added joint Torso_Leg5: type revolute, parent Torso, child Leg5, origin xyz=2 0 1 rpy=0 0 0, axis 1 0 0, limit lower=-3.14159 upper=3.14159 effort=0.0 velocity=0.0

File: body1002.urdf (robot description, URDF)
Before this commit: robot robot, 5 links, 4 joints
Links:
- added link Leg3, mass 1; collision box size=0.7164133264490005 1 1; visual box size=0.7164133264490005 1 1
- link Leg1: geometry collision box size=0.47445325062997884 1 1; visual box size=0.47445325062997884 1 1
- link Leg2: geometry collision box size=0.2719712417357227 1 1; visual box size=0.2719712417357227 1 1
- link Leg4: geometry collision box size=0.9603847710808506 1 1; visual box size=0.9603847710808506 1 1
- link Leg5: geometry collision box size=0.5687560502556714 1 1; visual box size=0.5687560502556714 1 1
Joints:
- added joint Torso_Leg3: type revolute, parent Torso, child Leg3, origin xyz=0.75 0 1 rpy=0 0 0, axis 1 0 0, limit lower=-3.14159 upper=3.14159 effort=0.0 velocity=0.0

File: body1003.urdf (robot description, URDF)
Before this commit: robot robot, 5 links, 4 joints
Links:
- removed link Leg3
- link Leg1: geometry collision box size=0.8130843537353594 1 1; visual box size=0.8130843537353594 1 1
- link Leg2: geometry collision box size=0.24731066352897885 1 1; visual box size=0.24731066352897885 1 1
- link Leg5: geometry collision box size=0.5946807773886 1 1; visual box size=0.5946807773886 1 1
Joints:
- removed joint Torso_Leg3

File: body1004.urdf (robot description, URDF)
Before this commit: robot robot, 6 links, 5 joints
Links:
- removed link Leg4
- link Leg1: geometry collision box size=0.38752043862213026 1 1; visual box size=0.38752043862213026 1 1
- link Leg2: geometry collision box size=0.45483681178305846 1 1; visual box size=0.45483681178305846 1 1
- link Leg3: geometry collision box size=0.640921333965637 1 1; visual box size=0.640921333965637 1 1
- link Leg5: geometry collision box size=0.8477133213128221 1 1; visual box size=0.8477133213128221 1 1
Joints:
- removed joint Torso_Leg4

File: body1005.urdf (robot description, URDF)
Before this commit: robot robot, 3 links, 2 joints
Links:
- added link Leg4, mass 1; collision box size=0.2984467891342999 1 1; visual box size=0.2984467891342999 1 1
- added link Leg5, mass 1; collision box size=0.31294934174659733 1 1; visual box size=0.31294934174659733 1 1
- link Leg1: geometry collision box size=0.914261018882869 1 1; visual box size=0.914261018882869 1 1
- link Leg2: geometry collision box size=0.7670915368310809 1 1; visual box size=0.7670915368310809 1 1
Joints:
- added joint Torso_Leg4: type revolute, parent Torso, child Leg4, origin xyz=0 0 1 rpy=0 0 0, axis 1 0 0, limit lower=-3.14159 upper=3.14159 effort=0.0 velocity=0.0
- added joint Torso_Leg5: type revolute, parent Torso, child Leg5, origin xyz=2 0 1 rpy=0 0 0, axis 1 0 0, limit lower=-3.14159 upper=3.14159 effort=0.0 velocity=0.0

File: body1006.urdf (robot description, URDF)
Before this commit: robot robot, 4 links, 3 joints
Links:
- removed link Leg4
- added link Leg2, mass 1; collision box size=0.5837454040120413 1 1; visual box size=0.5837454040120413 1 1
- added link Leg5, mass 1; collision box size=0.38728134584300905 1 1; visual box size=0.38728134584300905 1 1
- link Leg1: geometry collision box size=0.3112766648173696 1 1; visual box size=0.3112766648173696 1 1
- link Leg3: geometry collision box size=0.5902679135300102 1 1; visual box size=0.5902679135300102 1 1
Joints:
- removed joint Torso_Leg4
- added joint Torso_Leg2: type revolute, parent Torso, child Leg2, origin xyz=1.5 0 1 rpy=0 0 0, axis 1 0 0, limit lower=-3.14159 upper=3.14159 effort=0.0 velocity=0.0
- added joint Torso_Leg5: type revolute, parent Torso, child Leg5, origin xyz=2 0 1 rpy=0 0 0, axis 1 0 0, limit lower=-3.14159 upper=3.14159 effort=0.0 velocity=0.0

File: body1007.urdf (robot description, URDF)
Before this commit: robot robot, 6 links, 5 joints
Links:
- link Leg1: geometry collision box size=0.3852238434797549 1 1; visual box size=0.3852238434797549 1 1
- link Leg2: geometry collision box size=0.49951296545684515 1 1; visual box size=0.49951296545684515 1 1
- link Leg3: geometry collision box size=0.6427125713863681 1 1; visual box size=0.6427125713863681 1 1
- link Leg4: geometry collision box size=0.475657339129697 1 1; visual box size=0.475657339129697 1 1
- link Leg5: geometry collision box size=0.21908952520066327 1 1; visual box size=0.21908952520066327 1 1

File: body1008.urdf (robot description, URDF)
Before this commit: robot robot, 4 links, 3 joints
Links:
- removed link Leg5
- link Leg1: geometry collision box size=0.5160147992653115 1 1; visual box size=0.5160147992653115 1 1
- link Leg4: geometry collision box size=0.9133555536198807 1 1; visual box size=0.9133555536198807 1 1
Joints:
- removed joint Torso_Leg5

File: body1009.urdf (robot description, URDF)
Before this commit: robot robot, 5 links, 4 joints
Links:
- removed link Leg3
- removed link Leg4
- added link Leg2, mass 1; collision box size=0.31165876462032555 1 1; visual box size=0.31165876462032555 1 1
- link Leg1: geometry collision box size=0.7625929865404248 1 1; visual box size=0.7625929865404248 1 1
- link Leg5: geometry collision box size=0.7774540223581996 1 1; visual box size=0.7774540223581996 1 1
Joints:
- removed joint Torso_Leg3
- removed joint Torso_Leg4
- added joint Torso_Leg2: type revolute, parent Torso, child Leg2, origin xyz=1.5 0 1 rpy=0 0 0, axis 1 0 0, limit lower=-3.14159 upper=3.14159 effort=0.0 velocity=0.0

File: body101.urdf (robot description, URDF)
Before this commit: robot robot, 6 links, 5 joints
Links:
- removed link Leg4
- link Leg1: geometry collision box size=0.28396016229008136 1 1; visual box size=0.28396016229008136 1 1
- link Leg2: geometry collision box size=0.7637493143828797 1 1; visual box size=0.7637493143828797 1 1
- link Leg3: geometry collision box size=0.43566008639779885 1 1; visual box size=0.43566008639779885 1 1
- link Leg5: geometry collision box size=0.7685113083766879 1 1; visual box size=0.7685113083766879 1 1
Joints:
- removed joint Torso_Leg4

File: body102.urdf (robot description, URDF)
Before this commit: robot robot, 5 links, 4 joints
Links:
- removed link Leg3
- link Leg1: geometry collision box size=0.39215259982033673 1 1; visual box size=0.39215259982033673 1 1
- link Leg2: geometry collision box size=0.7800480426021181 1 1; visual box size=0.7800480426021181 1 1
- link Leg5: geometry collision box size=0.6121092600844067 1 1; visual box size=0.6121092600844067 1 1
Joints:
- removed joint Torso_Leg3

File: body103.urdf (robot description, URDF)
Before this commit: robot robot, 3 links, 2 joints
Links:
- added link Leg2, mass 1; collision box size=0.3864736318692111 1 1; visual box size=0.3864736318692111 1 1
- added link Leg3, mass 1; collision box size=0.8892982440032868 1 1; visual box size=0.8892982440032868 1 1
- added link Leg4, mass 1; collision box size=0.4824851608029887 1 1; visual box size=0.4824851608029887 1 1
- link Leg1: geometry collision box size=0.6277794044077416 1 1; visual box size=0.6277794044077416 1 1
- link Leg5: geometry collision box size=0.2871358400770884 1 1; visual box size=0.2871358400770884 1 1
Joints:
- added joint Torso_Leg2: type revolute, parent Torso, child Leg2, origin xyz=1.5 0 1 rpy=0 0 0, axis 1 0 0, limit lower=-3.14159 upper=3.14159 effort=0.0 velocity=0.0
- added joint Torso_Leg3: type revolute, parent Torso, child Leg3, origin xyz=0.75 0 1 rpy=0 0 0, axis 1 0 0, limit lower=-3.14159 upper=3.14159 effort=0.0 velocity=0.0
- added joint Torso_Leg4: type revolute, parent Torso, child Leg4, origin xyz=0 0 1 rpy=0 0 0, axis 1 0 0, limit lower=-3.14159 upper=3.14159 effort=0.0 velocity=0.0

File: body104.urdf (robot description, URDF)
Before this commit: robot robot, 3 links, 2 joints
Links:
- added link Leg2, mass 1; collision box size=0.5061891039819129 1 1; visual box size=0.5061891039819129 1 1
- added link Leg3, mass 1; collision box size=0.7134128997001985 1 1; visual box size=0.7134128997001985 1 1
- added link Leg5, mass 1; collision box size=0.830707979641572 1 1; visual box size=0.830707979641572 1 1
- link Leg1: geometry collision box size=0.7191857842425882 1 1; visual box size=0.7191857842425882 1 1
- link Leg4: geometry collision box size=0.9400854166480936 1 1; visual box size=0.9400854166480936 1 1
Joints:
- added joint Torso_Leg2: type revolute, parent Torso, child Leg2, origin xyz=1.5 0 1 rpy=0 0 0, axis 1 0 0, limit lower=-3.14159 upper=3.14159 effort=0.0 velocity=0.0
- added joint Torso_Leg3: type revolute, parent Torso, child Leg3, origin xyz=0.75 0 1 rpy=0 0 0, axis 1 0 0, limit lower=-3.14159 upper=3.14159 effort=0.0 velocity=0.0
- added joint Torso_Leg5: type revolute, parent Torso, child Leg5, origin xyz=2 0 1 rpy=0 0 0, axis 1 0 0, limit lower=-3.14159 upper=3.14159 effort=0.0 velocity=0.0

File: body105.urdf (robot description, URDF)
Before this commit: robot robot, 4 links, 3 joints
Links:
- added link Leg5, mass 1; collision box size=0.7713357773749487 1 1; visual box size=0.7713357773749487 1 1
- link Leg1: geometry collision box size=0.9206937840953695 1 1; visual box size=0.9206937840953695 1 1
- link Leg3: geometry collision box size=0.27063285115988855 1 1; visual box size=0.27063285115988855 1 1
- link Leg4: geometry collision box size=0.7777615913333684 1 1; visual box size=0.7777615913333684 1 1
Joints:
- added joint Torso_Leg5: type revolute, parent Torso, child Leg5, origin xyz=2 0 1 rpy=0 0 0, axis 1 0 0, limit lower=-3.14159 upper=3.14159 effort=0.0 velocity=0.0

File: body106.urdf (robot description, URDF)
Before this commit: robot robot, 6 links, 5 joints
Links:
- link Leg1: geometry collision box size=0.6637024882624029 1 1; visual box size=0.6637024882624029 1 1
- link Leg2: geometry collision box size=0.7150993372697891 1 1; visual box size=0.7150993372697891 1 1
- link Leg3: geometry collision box size=0.6923706800284659 1 1; visual box size=0.6923706800284659 1 1
- link Leg4: geometry collision box size=0.6259501897187385 1 1; visual box size=0.6259501897187385 1 1
- link Leg5: geometry collision box size=0.8700917587774497 1 1; visual box size=0.8700917587774497 1 1
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
Commit message: hm

File: body0.urdf (robot description, URDF)
Before this commit: robot robot, 6 links, 5 joints
Links:
- link Leg1: geometry collision box size=0.47453719015494533 1 1; visual box size=0.47453719015494533 1 1
- link Leg2: geometry collision box size=0.9562861561696689 1 1; visual box size=0.9562861561696689 1 1
- link Leg3: geometry collision box size=0.4184890685022925 1 1; visual box size=0.4184890685022925 1 1
- link Leg4: geometry collision box size=0.6522945038882819 1 1; visual box size=0.6522945038882819 1 1
- link Leg5: geometry collision box size=0.9907815974066436 1 1; visual box size=0.9907815974066436 1 1

File: body1.urdf (robot description, URDF)
Before this commit: robot robot, 3 links, 2 joints
Links:
- removed link Leg3
- added link Leg2, mass 1; collision box size=0.4406854469989576 1 1; visual box size=0.4406854469989576 1 1
- added link Leg4, mass 1; collision box size=0.9846530120448185 1 1; visual box size=0.9846530120448185 1 1
- added link Leg5, mass 1; collision box size=0.8287881332164808 1 1; visual box size=0.8287881332164808 1 1
- link Leg1: geometry collision box size=0.22912055170684342 1 1; visual box size=0.22912055170684342 1 1
Joints:
- removed joint Torso_Leg3
- added joint Torso_Leg2: type revolute, parent Torso, child Leg2, origin xyz=1.5 0 1 rpy=0 0 0, axis 1 0 0, limit lower=-3.14159 upper=3.14159 effort=0.0 velocity=0.0
- added joint Torso_Leg4: type revolute, parent Torso, child Leg4, origin xyz=0 0 1 rpy=0 0 0, axis 1 0 0, limit lower=-3.14159 upper=3.14159 effort=0.0 velocity=0.0
- added joint Torso_Leg5: type revolute, parent Torso, child Leg5, origin xyz=2 0 1 rpy=0 0 0, axis 1 0 0, limit lower=-3.14159 upper=3.14159 effort=0.0 velocity=0.0
