Commit message: not working

File: body1.urdf (robot description, URDF)
Before this commit: robot robot, 3 links, 2 joints
Links:
- removed link Leg1
- removed link Leg3
- removed link Torso
- added link Torso0, mass 1; collision box size=4 1 1; visual box size=4 1 1
- added link Torso0Leg1, mass 1; collision box size=0.6595365813614024 1 1; visual box size=0.6595365813614024 1 1
- added link Torso0Leg4, mass 1; collision box size=0.24559932749033397 1 1; visual box size=0.24559932749033397 1 1
- added link Torso0Leg5, mass 1; collision box size=0.67069293915625 1 1; visual box size=0.67069293915625 1 1
- added link Torso1, mass 1; collision box size=4 1 1; visual box size=4 1 1
- added link Torso1Leg1, mass 1; collision box size=0.8641143118767578 1 1; visual box size=0.8641143118767578 1 1
- added link Torso1Leg2, mass 1; collision box size=0.7696668931320909 1 1; visual box size=0.7696668931320909 1 1
- added link Torso1Leg4, mass 1; collision box size=0.5925592603272236 1 1; visual box size=0.5925592603272236 1 1
- added link Torso1Leg5, mass 1; collision box size=0.6984262867808344 1 1; visual box size=0.6984262867808344 1 1
Joints:
- removed joint Torso_Leg1
- removed joint Torso_Leg3
- added joint Torso0_Torso0Leg1: type revolute, parent Torso0, child Torso0Leg1, origin xyz=0.5 0 1 rpy=0 0 0, axis 1 0 0, limit lower=-3.14159 upper=3.14159 effort=0.0 velocity=0.0
- added joint Torso0_Torso0Leg4: type revolute, parent Torso0, child Torso0Leg4, origin xyz=0 0 1 rpy=0 0 0, axis 1 0 0, limit lower=-3.14159 upper=3.14159 effort=0.0 velocity=0.0
- added joint Torso0_Torso0Leg5: type revolute, parent Torso0, child Torso0Leg5, origin xyz=2 0 1 rpy=0 0 0, axis 1 0 0, limit lower=-3.14159 upper=3.14159 effort=0.0 velocity=0.0
- added joint Torso1_Torso0: type revolute, parent Torso1, child Torso0, origin xyz=0 4 0 rpy=0 0 0, axis 1 0 0, limit lower=-3.14159 upper=3.14159 effort=0.0 velocity=0.0
- added joint Torso1_Torso1Leg1: type revolute, parent Torso1, child Torso1Leg1, origin xyz=0.5 0 1 rpy=0 0 0, axis 1 0 0, limit lower=-3.14159 upper=3.14159 effort=0.0 velocity=0.0
- added joint Torso1_Torso1Leg2: type revolute, parent Torso1, child Torso1Leg2, origin xyz=1.5 0 1 rpy=0 0 0, axis 1 0 0, limit lower=-3.14159 upper=3.14159 effort=0.0 velocity=0.0
- added joint Torso1_Torso1Leg4: type revolute, parent Torso1, child Torso1Leg4, origin xyz=0 0 1 rpy=0 0 0, axis 1 0 0, limit lower=-3.14159 upper=3.14159 effort=0.0 velocity=0.0
- added joint Torso1_Torso1Leg5: type revolute, parent Torso1, child Torso1Leg5, origin xyz=2 0 1 rpy=0 0 0, axis 1 0 0, limit lower=-3.14159 upper=3.14159 effort=0.0 velocity=0.0

File: body2.urdf (robot description, URDF)
Before this commit: robot robot, 12 links, 11 joints
Links:
- removed link Torso0Leg3
- removed link Torso1Leg2
- removed link Torso1Leg3
- removed link Torso1Leg5
- link Torso0Leg1: geometry collision box size=0.47812749204272137 1 1; visual box size=0.47812749204272137 1 1
- link Torso0Leg2: geometry collision box size=0.731075837349821 1 1; visual box size=0.731075837349821 1 1
- link Torso0Leg4: geometry collision box size=0.37194177606853807 1 1; visual box size=0.37194177606853807 1 1
- link Torso0Leg5: geometry collision box size=0.8288388887732148 1 1; visual box size=0.8288388887732148 1 1
- link Torso1Leg1: geometry collision box size=0.6455313501635533 1 1; visual box size=0.6455313501635533 1 1
- link Torso1Leg4: geometry collision box size=0.8881197884961436 1 1; visual box size=0.8881197884961436 1 1
Joints:
- removed joint Torso0_Torso0Leg3
- removed joint Torso1_Torso1Leg2
- removed joint Torso1_Torso1Leg3
- removed joint Torso1_Torso1Leg5

File: body3.urdf (robot description, URDF)
Before this commit: robot robot, 12 links, 11 joints
Links:
- removed link Torso0Leg2
- removed link Torso0Leg3
- removed link Torso0Leg4
- removed link Torso1Leg5
- link Torso0Leg1: geometry collision box size=0.230119286102269 1 1; visual box size=0.230119286102269 1 1
- link Torso0Leg5: geometry collision box size=0.5997879213224315 1 1; visual box size=0.5997879213224315 1 1
- link Torso1Leg1: geometry collision box size=0.21102195261173806 1 1; visual box size=0.21102195261173806 1 1
- link Torso1Leg2: geometry collision box size=0.5177203848302916 1 1; visual box size=0.5177203848302916 1 1
- link Torso1Leg3: geometry collision box size=0.670090166889048 1 1; visual box size=0.670090166889048 1 1
- link Torso1Leg4: geometry collision box size=0.6970641411418084 1 1; visual box size=0.6970641411418084 1 1
Joints:
- removed joint Torso0_Torso0Leg2
- removed joint Torso0_Torso0Leg3
- removed joint Torso0_Torso0Leg4
- removed joint Torso1_Torso1Leg5

File: body4.urdf (robot description, URDF)
Before this commit: robot robot, 12 links, 11 joints
Links:
- removed link Torso0Leg4
- removed link Torso1Leg3
- removed link Torso1Leg5
- link Torso0Leg1: geometry collision box size=0.5381811430341946 1 1; visual box size=0.5381811430341946 1 1
- link Torso0Leg2: geometry collision box size=0.24975467367338686 1 1; visual box size=0.24975467367338686 1 1
- link Torso0Leg3: geometry collision box size=0.9960176754775214 1 1; visual box size=0.9960176754775214 1 1
- link Torso0Leg5: geometry collision box size=0.5201716842271491 1 1; visual box size=0.5201716842271491 1 1
- link Torso1Leg1: geometry collision box size=0.713736848724658 1 1; visual box size=0.713736848724658 1 1
- link Torso1Leg2: geometry collision box size=0.49605478257826974 1 1; visual box size=0.49605478257826974 1 1
- link Torso1Leg4: geometry collision box size=0.5164878030918523 1 1; visual box size=0.5164878030918523 1 1
Joints:
- removed joint Torso0_Torso0Leg4
- removed joint Torso1_Torso1Leg3
- removed joint Torso1_Torso1Leg5

File: body5.urdf (robot description, URDF)
Before this commit: robot robot, 12 links, 11 joints
Links:
- removed link Torso0Leg2
- removed link Torso0Leg3
- removed link Torso0Leg4
- removed link Torso1Leg5
- link Torso0Leg1: geometry collision box size=0.8076302422886263 1 1; visual box size=0.8076302422886263 1 1
- link Torso0Leg5: geometry collision box size=0.3990754818700377 1 1; visual box size=0.3990754818700377 1 1
- link Torso1Leg1: geometry collision box size=0.6299320362317959 1 1; visual box size=0.6299320362317959 1 1
- link Torso1Leg2: geometry collision box size=0.7606741164624236 1 1; visual box size=0.7606741164624236 1 1
- link Torso1Leg3: geometry collision box size=0.4411297895735671 1 1; visual box size=0.4411297895735671 1 1
- link Torso1Leg4: geometry collision box size=0.3132216523326812 1 1; visual box size=0.3132216523326812 1 1
Joints:
- removed joint Torso0_Torso0Leg2
- removed joint Torso0_Torso0Leg3
- removed joint Torso0_Torso0Leg4
- removed joint Torso1_Torso1Leg5
