Commit message: final wo rking

File: body/body0.urdf (robot description, URDF)
Before this commit: robot robot, 5 links, 4 joints
Links:
- removed link Torso0Leg3
- removed link Torso0Leg4
- removed link Torso0Leg5
- added link Torso0Leg2, mass 1; collision box size=0.9605763633912052 1 1; visual box size=0.9605763633912052 1 1
- link Torso0Leg1: geometry collision box size=0.3256601081005355 1 1; visual box size=0.3256601081005355 1 1
Joints:
- removed joint Torso0_Torso0Leg3
- removed joint Torso0_Torso0Leg4
- removed joint Torso0_Torso0Leg5
- added joint Torso0_Torso0Leg2: type revolute, parent Torso0, child Torso0Leg2, origin xyz=1.5 0 1 rpy=0 0 0, axis 1 0 0, limit lower=-3.14159 upper=3.14159 effort=0.0 velocity=0.0

File: body/body1.urdf (robot description, URDF)
Before this commit: robot robot, 3 links, 2 joints
Links:
- added link Torso0Leg2, mass 1; collision box size=0.8001691686781829 1 1; visual box size=0.8001691686781829 1 1
- link Torso0Leg1: geometry collision box size=0.3762575907029419 1 1; visual box size=0.3762575907029419 1 1
- link Torso0Leg5: geometry collision box size=0.49272695130816246 1 1; visual box size=0.49272695130816246 1 1
Joints:
- added joint Torso0_Torso0Leg2: type revolute, parent Torso0, child Torso0Leg2, origin xyz=1.5 0 1 rpy=0 0 0, axis 1 0 0, limit lower=-3.14159 upper=3.14159 effort=0.0 velocity=0.0

File: body/body10.urdf (robot description, URDF)
Before this commit: robot robot, 6 links, 5 joints
Links:
- link Torso0Leg1: geometry collision box size=0.48908149998655265 1 1; visual box size=0.48908149998655265 1 1
- link Torso0Leg2: geometry collision box size=0.41396984338361753 1 1; visual box size=0.41396984338361753 1 1
- link Torso0Leg3: geometry collision box size=0.9202368492989002 1 1; visual box size=0.9202368492989002 1 1
- link Torso0Leg4: geometry collision box size=0.5936636919280517 1 1; visual box size=0.5936636919280517 1 1
- link Torso0Leg5: geometry collision box size=0.33469704613136886 1 1; visual box size=0.33469704613136886 1 1

File: body/body11.urdf (robot description, URDF)
Before this commit: robot robot, 4 links, 3 joints
Links:
- added link Torso0Leg4, mass 1; collision box size=0.48691045596716354 1 1; visual box size=0.48691045596716354 1 1
- added link Torso0Leg5, mass 1; collision box size=0.20945723281345183 1 1; visual box size=0.20945723281345183 1 1
- link Torso0Leg1: geometry collision box size=0.461990380485199 1 1; visual box size=0.461990380485199 1 1
- link Torso0Leg2: geometry collision box size=0.5867278860165419 1 1; visual box size=0.5867278860165419 1 1
- link Torso0Leg3: geometry collision box size=0.4625771219034044 1 1; visual box size=0.4625771219034044 1 1
Joints:
- added joint Torso0_Torso0Leg4: type revolute, parent Torso0, child Torso0Leg4, origin xyz=0 0 1 rpy=0 0 0, axis 1 0 0, limit lower=-3.14159 upper=3.14159 effort=0.0 velocity=0.0
- added joint Torso0_Torso0Leg5: type revolute, parent Torso0, child Torso0Leg5, origin xyz=2 0 1 rpy=0 0 0, axis 1 0 0, limit lower=-3.14159 upper=3.14159 effort=0.0 velocity=0.0

File: body/body12.urdf (robot description, URDF)
Before this commit: robot robot, 6 links, 5 joints
Links:
- removed link Torso0Leg2
- removed link Torso0Leg3
- removed link Torso0Leg4
- link Torso0Leg1: geometry collision box size=0.43714332661449967 1 1; visual box size=0.43714332661449967 1 1
- link Torso0Leg5: geometry collision box size=0.674895580693392 1 1; visual box size=0.674895580693392 1 1
Joints:
- removed joint Torso0_Torso0Leg2
- removed joint Torso0_Torso0Leg3
- removed joint Torso0_Torso0Leg4

File: body/body13.urdf (robot description, URDF)
Before this commit: robot robot, 6 links, 5 joints
Links:
- link Torso0Leg1: geometry collision box size=0.2987385672549545 1 1; visual box size=0.2987385672549545 1 1
- link Torso0Leg2: geometry collision box size=0.8391158958389788 1 1; visual box size=0.8391158958389788 1 1
- link Torso0Leg3: geometry collision box size=0.4935631544724781 1 1; visual box size=0.4935631544724781 1 1
- link Torso0Leg4: geometry collision box size=0.4256680729522646 1 1; visual box size=0.4256680729522646 1 1
- link Torso0Leg5: geometry collision box size=0.7421811722917668 1 1; visual box size=0.7421811722917668 1 1

File: body/body14.urdf (robot description, URDF)
Before this commit: robot robot, 4 links, 3 joints
Links:
- added link Torso0Leg3, mass 1; collision box size=0.3138801803009071 1 1; visual box size=0.3138801803009071 1 1
- added link Torso0Leg4, mass 1; collision box size=0.7999641148704117 1 1; visual box size=0.7999641148704117 1 1
- link Torso0Leg1: geometry collision box size=0.7113199132301906 1 1; visual box size=0.7113199132301906 1 1
- link Torso0Leg2: geometry collision box size=0.30818064709711995 1 1; visual box size=0.30818064709711995 1 1
- link Torso0Leg5: geometry collision box size=0.20222792414234736 1 1; visual box size=0.20222792414234736 1 1
Joints:
- added joint Torso0_Torso0Leg3: type revolute, parent Torso0, child Torso0Leg3, origin xyz=0.75 0 1 rpy=0 0 0, axis 1 0 0, limit lower=-3.14159 upper=3.14159 effort=0.0 velocity=0.0
- added joint Torso0_Torso0Leg4: type revolute, parent Torso0, child Torso0Leg4, origin xyz=0 0 1 rpy=0 0 0, axis 1 0 0, limit lower=-3.14159 upper=3.14159 effort=0.0 velocity=0.0

File: body/body15.urdf (robot description, URDF)
Before this commit: robot robot, 5 links, 4 joints
Links:
- removed link Torso0Leg4
- removed link Torso0Leg5
- added link Torso0Leg3, mass 1; collision box size=0.39469994736204167 1 1; visual box size=0.39469994736204167 1 1
- link Torso0Leg1: geometry collision box size=0.5930129775877089 1 1; visual box size=0.5930129775877089 1 1
- link Torso0Leg2: geometry collision box size=0.4056939482315192 1 1; visual box size=0.4056939482315192 1 1
Joints:
- removed joint Torso0_Torso0Leg4
- removed joint Torso0_Torso0Leg5
- added joint Torso0_Torso0Leg3: type revolute, parent Torso0, child Torso0Leg3, origin xyz=0.75 0 1 rpy=0 0 0, axis 1 0 0, limit lower=-3.14159 upper=3.14159 effort=0.0 velocity=0.0

File: body/body16.urdf (robot description, URDF)
Before this commit: robot robot, 3 links, 2 joints
Links:
- removed link Torso0Leg2
- added link Torso0Leg4, mass 1; collision box size=0.8008899679060104 1 1; visual box size=0.8008899679060104 1 1
- link Torso0Leg1: geometry collision box size=0.5382213039265649 1 1; visual box size=0.5382213039265649 1 1
Joints:
- removed joint Torso0_Torso0Leg2
- added joint Torso0_Torso0Leg4: type revolute, parent Torso0, child Torso0Leg4, origin xyz=0 0 1 rpy=0 0 0, axis 1 0 0, limit lower=-3.14159 upper=3.14159 effort=0.0 velocity=0.0

File: body/body17.urdf (robot description, URDF)
Before this commit: robot robot, 3 links, 2 joints
Links:
- added link Torso0Leg2, mass 1; collision box size=0.27265237182855195 1 1; visual box size=0.27265237182855195 1 1
- link Torso0Leg1: geometry collision box size=0.5871767461247802 1 1; visual box size=0.5871767461247802 1 1
- link Torso0Leg3: geometry collision box size=0.8653242144719988 1 1; visual box size=0.8653242144719988 1 1
Joints:
- added joint Torso0_Torso0Leg2: type revolute, parent Torso0, child Torso0Leg2, origin xyz=1.5 0 1 rpy=0 0 0, axis 1 0 0, limit lower=-3.14159 upper=3.14159 effort=0.0 velocity=0.0

File: body/body18.urdf (robot description, URDF)
Before this commit: robot robot, 4 links, 3 joints
Links:
- added link Torso0Leg3, mass 1; collision box size=0.8272661938877948 1 1; visual box size=0.8272661938877948 1 1
- link Torso0Leg1: geometry collision box size=0.7203362320608806 1 1; visual box size=0.7203362320608806 1 1
- link Torso0Leg2: geometry collision box size=0.7899973231504143 1 1; visual box size=0.7899973231504143 1 1
- link Torso0Leg5: geometry collision box size=0.9500378432088039 1 1; visual box size=0.9500378432088039 1 1
Joints:
- added joint Torso0_Torso0Leg3: type revolute, parent Torso0, child Torso0Leg3, origin xyz=0.75 0 1 rpy=0 0 0, axis 1 0 0, limit lower=-3.14159 upper=3.14159 effort=0.0 velocity=0.0

File: body/body19.urdf (robot description, URDF)
Before this commit: robot robot, 4 links, 3 joints
Links:
- removed link Torso0Leg3
- added link Torso0Leg2, mass 1; collision box size=0.7631075276942656 1 1; visual box size=0.7631075276942656 1 1
- added link Torso0Leg5, mass 1; collision box size=0.32317905758544896 1 1; visual box size=0.32317905758544896 1 1
- link Torso0Leg1: geometry collision box size=0.21392373778419282 1 1; visual box size=0.21392373778419282 1 1
- link Torso0Leg4: geometry collision box size=0.4275885019888486 1 1; visual box size=0.4275885019888486 1 1
Joints:
- removed joint Torso0_Torso0Leg3
- added joint Torso0_Torso0Leg2: type revolute, parent Torso0, child Torso0Leg2, origin xyz=1.5 0 1 rpy=0 0 0, axis 1 0 0, limit lower=-3.14159 upper=3.14159 effort=0.0 velocity=0.0
- added joint Torso0_Torso0Leg5: type revolute, parent Torso0, child Torso0Leg5, origin xyz=2 0 1 rpy=0 0 0, axis 1 0 0, limit lower=-3.14159 upper=3.14159 effort=0.0 velocity=0.0

File: body/body2.urdf (robot description, URDF)
Before this commit: robot robot, 4 links, 3 joints
Links:
- added link Torso0Leg4, mass 1; collision box size=0.5812853337028552 1 1; visual box size=0.5812853337028552 1 1
- added link Torso0Leg5, mass 1; collision box size=0.26101878699058667 1 1; visual box size=0.26101878699058667 1 1
- link Torso0Leg1: geometry collision box size=0.9646001064634013 1 1; visual box size=0.9646001064634013 1 1
- link Torso0Leg2: geometry collision box size=0.6775954579866733 1 1; visual box size=0.6775954579866733 1 1
- link Torso0Leg3: geometry collision box size=0.6644828548027706 1 1; visual box size=0.6644828548027706 1 1
Joints:
- added joint Torso0_Torso0Leg4: type revolute, parent Torso0, child Torso0Leg4, origin xyz=0 0 1 rpy=0 0 0, axis 1 0 0, limit lower=-3.14159 upper=3.14159 effort=0.0 velocity=0.0
- added joint Torso0_Torso0Leg5: type revolute, parent Torso0, child Torso0Leg5, origin xyz=2 0 1 rpy=0 0 0, axis 1 0 0, limit lower=-3.14159 upper=3.14159 effort=0.0 velocity=0.0

File: body/body3.urdf (robot description, URDF)
Before this commit: robot robot, 3 links, 2 joints
Links:
- added link Torso0Leg2, mass 1; collision box size=0.6776212093136584 1 1; visual box size=0.6776212093136584 1 1
- added link Torso0Leg3, mass 1; collision box size=0.5867630688348414 1 1; visual box size=0.5867630688348414 1 1
- added link Torso0Leg4, mass 1; collision box size=0.4720693959248965 1 1; visual box size=0.4720693959248965 1 1
- link Torso0Leg1: geometry collision box size=0.8027797423851106 1 1; visual box size=0.8027797423851106 1 1
- link Torso0Leg5: geometry collision box size=0.5944862624451519 1 1; visual box size=0.5944862624451519 1 1
Joints:
- added joint Torso0_Torso0Leg2: type revolute, parent Torso0, child Torso0Leg2, origin xyz=1.5 0 1 rpy=0 0 0, axis 1 0 0, limit lower=-3.14159 upper=3.14159 effort=0.0 velocity=0.0
- added joint Torso0_Torso0Leg3: type revolute, parent Torso0, child Torso0Leg3, origin xyz=0.75 0 1 rpy=0 0 0, axis 1 0 0, limit lower=-3.14159 upper=3.14159 effort=0.0 velocity=0.0
- added joint Torso0_Torso0Leg4: type revolute, parent Torso0, child Torso0Leg4, origin xyz=0 0 1 rpy=0 0 0, axis 1 0 0, limit lower=-3.14159 upper=3.14159 effort=0.0 velocity=0.0

File: body/body4.urdf (robot description, URDF)
Before this commit: robot robot, 6 links, 5 joints
Links:
- removed link Torso0Leg4
- link Torso0Leg1: geometry collision box size=0.22629538140186725 1 1; visual box size=0.22629538140186725 1 1
- link Torso0Leg2: geometry collision box size=0.6090037155490111 1 1; visual box size=0.6090037155490111 1 1
- link Torso0Leg3: geometry collision box size=0.7350987196923771 1 1; visual box size=0.7350987196923771 1 1
- link Torso0Leg5: geometry collision box size=0.9802798438380258 1 1; visual box size=0.9802798438380258 1 1
Joints:
- removed joint Torso0_Torso0Leg4

File: body/body5.urdf (robot description, URDF)
Before this commit: robot robot, 6 links, 5 joints
Links:
- removed link Torso0Leg2
- link Torso0Leg1: geometry collision box size=0.7539756528251222 1 1; visual box size=0.7539756528251222 1 1
- link Torso0Leg3: geometry collision box size=0.38793999959534997 1 1; visual box size=0.38793999959534997 1 1
- link Torso0Leg4: geometry collision box size=0.6690452825455889 1 1; visual box size=0.6690452825455889 1 1
- link Torso0Leg5: geometry collision box size=0.45349403385658893 1 1; visual box size=0.45349403385658893 1 1
Joints:
- removed joint Torso0_Torso0Leg2

File: body/body6.urdf (robot description, URDF)
Before this commit: robot robot, 5 links, 4 joints
Links:
- added link Torso0Leg4, mass 1; collision box size=0.28175842536815393 1 1; visual box size=0.28175842536815393 1 1
- link Torso0Leg1: geometry collision box size=0.8538016605775209 1 1; visual box size=0.8538016605775209 1 1
- link Torso0Leg2: geometry collision box size=0.8496302200141512 1 1; visual box size=0.8496302200141512 1 1
- link Torso0Leg3: geometry collision box size=0.8594007199180067 1 1; visual box size=0.8594007199180067 1 1
- link Torso0Leg5: geometry collision box size=0.26082002064244386 1 1; visual box size=0.26082002064244386 1 1
Joints:
- added joint Torso0_Torso0Leg4: type revolute, parent Torso0, child Torso0Leg4, origin xyz=0 0 1 rpy=0 0 0, axis 1 0 0, limit lower=-3.14159 upper=3.14159 effort=0.0 velocity=0.0

File: body/body7.urdf (robot description, URDF)
Before this commit: robot robot, 3 links, 2 joints
Links:
- removed link Torso0Leg5
- added link Torso0Leg4, mass 1; collision box size=0.9417356314152634 1 1; visual box size=0.9417356314152634 1 1
- link Torso0Leg1: geometry collision box size=0.46894164677387185 1 1; visual box size=0.46894164677387185 1 1
Joints:
- removed joint Torso0_Torso0Leg5
- added joint Torso0_Torso0Leg4: type revolute, parent Torso0, child Torso0Leg4, origin xyz=0 0 1 rpy=0 0 0, axis 1 0 0, limit lower=-3.14159 upper=3.14159 effort=0.0 velocity=0.0

File: body/body8.urdf (robot description, URDF)
Before this commit: robot robot, 5 links, 4 joints
Links:
- removed link Torso0Leg3
- added link Torso0Leg2, mass 1; collision box size=0.9000403299423938 1 1; visual box size=0.9000403299423938 1 1
- link Torso0Leg1: geometry collision box size=0.36704063079771454 1 1; visual box size=0.36704063079771454 1 1
- link Torso0Leg4: geometry collision box size=0.8385580762135991 1 1; visual box size=0.8385580762135991 1 1
- link Torso0Leg5: geometry collision box size=0.31356350362165525 1 1; visual box size=0.31356350362165525 1 1
Joints:
- removed joint Torso0_Torso0Leg3
- added joint Torso0_Torso0Leg2: type revolute, parent Torso0, child Torso0Leg2, origin xyz=1.5 0 1 rpy=0 0 0, axis 1 0 0, limit lower=-3.14159 upper=3.14159 effort=0.0 velocity=0.0

File: body/body9.urdf (robot description, URDF)
Before this commit: robot robot, 5 links, 4 joints
Links:
- removed link Torso0Leg3
- removed link Torso0Leg4
- removed link Torso0Leg5
- added link Torso0Leg2, mass 1; collision box size=0.8416775784653177 1 1; visual box size=0.8416775784653177 1 1
- link Torso0Leg1: geometry collision box size=0.9266970836270589 1 1; visual box size=0.9266970836270589 1 1
Joints:
- removed joint Torso0_Torso0Leg3
- removed joint Torso0_Torso0Leg4
- removed joint Torso0_Torso0Leg5
- added joint Torso0_Torso0Leg2: type revolute, parent Torso0, child Torso0Leg2, origin xyz=1.5 0 1 rpy=0 0 0, axis 1 0 0, limit lower=-3.14159 upper=3.14159 effort=0.0 velocity=0.0
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
Commit message: readme

File: body/body0.urdf (robot description, URDF)
Before this commit: robot robot, 3 links, 2 joints
Links:
- added link Torso0Leg3, mass 1; collision box size=0.5164110540308495 1 1; visual box size=0.5164110540308495 1 1
- added link Torso0Leg4, mass 1; collision box size=0.5550646931936851 1 1; visual box size=0.5550646931936851 1 1
- added link Torso0Leg5, mass 1; collision box size=0.5781421423987428 1 1; visual box size=0.5781421423987428 1 1
- link Torso0Leg1: geometry collision box size=0.510417833763464 1 1; visual box size=0.510417833763464 1 1
- link Torso0Leg2: geometry collision box size=0.3570051234229024 1 1; visual box size=0.3570051234229024 1 1
Joints:
- added joint Torso0_Torso0Leg3: type revolute, parent Torso0, child Torso0Leg3, origin xyz=0.75 0 1 rpy=0 0 0, axis 1 0 0, limit lower=-3.14159 upper=3.14159 effort=0.0 velocity=0.0
- added joint Torso0_Torso0Leg4: type revolute, parent Torso0, child Torso0Leg4, origin xyz=0 0 1 rpy=0 0 0, axis 1 0 0, limit lower=-3.14159 upper=3.14159 effort=0.0 velocity=0.0
- added joint Torso0_Torso0Leg5: type revolute, parent Torso0, child Torso0Leg5, origin xyz=2 0 1 rpy=0 0 0, axis 1 0 0, limit lower=-3.14159 upper=3.14159 effort=0.0 velocity=0.0

File: body/body1.urdf (robot description, URDF)
Before this commit: robot robot, 4 links, 3 joints
Links:
- removed link Torso0Leg5
- added link Torso0Leg3, mass 1; collision box size=0.6529513403018188 1 1; visual box size=0.6529513403018188 1 1
- added link Torso0Leg4, mass 1; collision box size=0.6568852811692071 1 1; visual box size=0.6568852811692071 1 1
- link Torso0Leg1: geometry collision box size=0.8274479456534214 1 1; visual box size=0.8274479456534214 1 1
- link Torso0Leg2: geometry collision box size=0.7364043044688444 1 1; visual box size=0.7364043044688444 1 1
Joints:
- removed joint Torso0_Torso0Leg5
- added joint Torso0_Torso0Leg3: type revolute, parent Torso0, child Torso0Leg3, origin xyz=0.75 0 1 rpy=0 0 0, axis 1 0 0, limit lower=-3.14159 upper=3.14159 effort=0.0 velocity=0.0
- added joint Torso0_Torso0Leg4: type revolute, parent Torso0, child Torso0Leg4, origin xyz=0 0 1 rpy=0 0 0, axis 1 0 0, limit lower=-3.14159 upper=3.14159 effort=0.0 velocity=0.0

File: body/body2.urdf (robot description, URDF)
Before this commit: robot robot, 6 links, 5 joints
Links:
- removed link Torso0Leg2
- removed link Torso0Leg4
- link Torso0Leg1: geometry collision box size=0.8774235442122802 1 1; visual box size=0.8774235442122802 1 1
- link Torso0Leg3: geometry collision box size=0.496899366331387 1 1; visual box size=0.496899366331387 1 1
- link Torso0Leg5: geometry collision box size=0.4465126337828581 1 1; visual box size=0.4465126337828581 1 1
Joints:
- removed joint Torso0_Torso0Leg2
- removed joint Torso0_Torso0Leg4

File: body/body3.urdf (robot description, URDF)
Before this commit: robot robot, 6 links, 5 joints
Links:
- removed link Torso0Leg2
- removed link Torso0Leg3
- removed link Torso0Leg5
- link Torso0Leg1: geometry collision box size=0.7250171708760871 1 1; visual box size=0.7250171708760871 1 1
- link Torso0Leg4: geometry collision box size=0.2761670445603015 1 1; visual box size=0.2761670445603015 1 1
Joints:
- removed joint Torso0_Torso0Leg2
- removed joint Torso0_Torso0Leg3
- removed joint Torso0_Torso0Leg5
